File: PCB/stm_proto_board/stm_proto_board.kicad_pcb (KiCad board)
At the start: 2 copper layers, 2 parts, among them U1 STM32F103C8T6, U4 MCP2551-I-P

Commit message: Update PCB proto-board
Parts:
- added C1: CAP, Capacitor_SMD:CP_Elec_5x4.5, F.Cu at (53.3, 144.8)
- added C2: CAP, Capacitor_SMD:CP_Elec_5x4.5, F.Cu at (57.1, 137.2)
- added D1: D_Bridge_+-AA, Diode_THT:Diode_Bridge_DIP-4_W7.62mm_P5.08mm, F.Cu at (54.6, 114.3)
- added J1: Conn_01x08, Connector_PinHeader_2.54mm:PinHeader_1x08_P2.54mm_Vertical, F.Cu at (73.7, 121.9)
- added J11: Conn_01x04, Connector_PinHeader_2.54mm:PinHeader_1x04_P2.54mm_Vertical, F.Cu at (119.4, 113.0)
- added J12: Conn_01x04, Connector_PinHeader_2.54mm:PinHeader_1x04_P2.54mm_Vertical, F.Cu at (154.9, 137.2)
- added J13: Conn_01x04, Connector_PinHeader_2.54mm:PinHeader_1x04_P2.54mm_Vertical, F.Cu at (170.2, 144.8)
- added J14: Conn_01x08, Connector_PinHeader_2.54mm:PinHeader_1x08_P2.54mm_Vertical, F.Cu at (73.7, 144.8)
- added J15: Conn_01x02, Connector_PinHeader_2.54mm:PinHeader_1x02_P2.54mm_Vertical, F.Cu at (47.0, 109.2)
- added J2: Conn_01x04, Connector_PinHeader_2.54mm:PinHeader_1x04_P2.54mm_Horizontal, F.Cu at (47.0, 99.1)
- added J3: DB9_Female, Connector_Dsub:DSUB-9_Female_Horizontal_P2.77x2.84mm_EdgePinOffset4.94mm_Housed_MountingHolesOffset7.48mm, F.Cu at (181.6, 129.5)
- added J4: Conn_01x02, Connector_PinHeader_2.54mm:PinHeader_1x02_P2.54mm_Vertical, F.Cu at (170.2, 125.7)
- added J5: Conn_01x04, Connector_PinHeader_2.54mm:PinHeader_1x04_P2.54mm_Vertical, F.Cu at (119.4, 118.1)
- added J6: Conn_01x02, Connector_PinHeader_2.54mm:PinHeader_1x02_P2.54mm_Vertical, F.Cu at (194.3, 111.8)
- added J7: Conn_01x04, Connector_PinHeader_2.54mm:PinHeader_1x04_P2.54mm_Vertical, F.Cu at (194.3, 95.2)
- added R1: R, Resistor_THT:R_Axial_DIN0204_L3.6mm_D1.6mm_P7.62mm_Horizontal, F.Cu at (135.9, 124.5)
- added R10: 330, Resistor_THT:R_Axial_DIN0204_L3.6mm_D1.6mm_P7.62mm_Horizontal, F.Cu at (170.2, 113.0)
- added R2: R, Resistor_THT:R_Axial_DIN0204_L3.6mm_D1.6mm_P7.62mm_Horizontal, F.Cu at (135.9, 128.3)
- added R3: R, Resistor_THT:R_Axial_DIN0204_L3.6mm_D1.6mm_P7.62mm_Horizontal, F.Cu at (115.6, 128.3)
- added R4: R, Resistor_THT:R_Axial_DIN0204_L3.6mm_D1.6mm_P7.62mm_Horizontal, F.Cu at (115.6, 124.5)
- added R5: 10k, Resistor_THT:R_Axial_DIN0204_L3.6mm_D1.6mm_P7.62mm_Horizontal, F.Cu at (161.3, 128.3)
- added R6: 1.2k, Resistor_THT:R_Axial_DIN0204_L3.6mm_D1.6mm_P7.62mm_Horizontal, F.Cu at (77.5, 95.2)
- added R7: 330, Resistor_THT:R_Axial_DIN0204_L3.6mm_D1.6mm_P7.62mm_Horizontal, F.Cu at (152.4, 113.0)
- added R8: 330, Resistor_THT:R_Axial_DIN0204_L3.6mm_D1.6mm_P7.62mm_Horizontal, F.Cu at (152.4, 101.6)
- added R9: 330, Resistor_THT:R_Axial_DIN0204_L3.6mm_D1.6mm_P7.62mm_Horizontal, F.Cu at (170.2, 101.6)
- added SW1: SW_Push, Button_Switch_THT:SW_PUSH_6mm, F.Cu at (121.9, 143.5)
- added SW2: SW_Push, Button_Switch_THT:SW_PUSH_6mm, F.Cu at (141.0, 138.4)
- added SW3: SW_Push, Button_Switch_THT:SW_PUSH_6mm, F.Cu at (128.3, 129.5)
- added SW4: SW_Push, Button_Switch_THT:SW_PUSH_6mm, F.Cu at (115.6, 138.4)
- added U4: LTV-814, Package_DIP:DIP-4_W7.62mm, F.Cu at (161.3, 124.5)
- added U5: L7805, Package_TO_SOT_THT:TO-220-3_Vertical, F.Cu at (52.1, 128.3)
- added U6: 4N25, Package_DIP:DIP-6_W7.62mm, F.Cu at (156.2, 108.0)
- added U7: 4N25, Package_DIP:DIP-6_W7.62mm, F.Cu at (156.2, 96.5)
- added U8: 4N25, Package_DIP:DIP-6_W7.62mm, F.Cu at (174.0, 96.5)
- added U9: 4N25, Package_DIP:DIP-6_W7.62mm, F.Cu at (174.0, 108.0)
- U1: value STM32F103C8T6 -> YAAJ_BluePill_Part_Like; footprint Package_QFP:LQFP-48_7x7mm_P0.5mm -> Footprints:YAAJ_BluePill_1
- moved U2 83.7 mm to (61.0, 99.1), turned to 180 degrees
- moved U1 57.3 mm to (73.7, 105.4), turned to 90 degrees
- renumbered U4 to U2
Connections:
- net Net-(U1-Pad10) renamed Ext4
- net Net-(U1-Pad12) renamed Ext5
- net Net-(U1-Pad14) renamed Ext6
- net Net-(U1-Pad15) renamed Ext7
- net Net-(U1-Pad29) renamed Ext9
- net Net-(U1-Pad34) renamed Ext11
- net Net-(U1-Pad5) renamed Ext1
- net Net-(U1-Pad6) renamed Ext2
- net Net-(U1-Pad7) renamed Ext3
- U1 pad 1: Net-(U1-Pad1) -> /LCD_RST
- U1 pad 11: Net-(U1-Pad11) -> /LCD_CLK
- U1 pad 13: Net-(U1-Pad13) -> CAN_EN
- U1 pad 16: Net-(U1-Pad16) -> SCL
- U1 pad 17: Net-(U1-Pad17) -> SDA
- U1 pad 18: Net-(U1-Pad18) -> +5V
- U1 pad 19: Net-(U1-Pad19) -> GND
- U1 pad 2: Net-(U1-Pad2) -> /LCD_CE
- U1 pad 20: Net-(U1-Pad20) -> +3V3
- U1 pad 22: Net-(U1-Pad22) -> SW_UP
- U1 pad 23: Net-(U1-Pad23) -> SW_DOWN
- U1 pad 24: +3V3 -> SW_RIGHT
- U1 pad 25: /LCD_RST -> SW_LEFT
- U1 pad 26: /LCD_CE -> Ext8
- U1 pad 27: /LCD_DC -> USART2_TX
- U1 pad 28: /LCD_DIN -> USART2_RX
- U1 pad 3: Net-(U1-Pad3) -> /LCD_DC
- U1 pad 30: Net-(U1-Pad30) -> LED_W
- U1 pad 31: Net-(U1-Pad31) -> LED_B
- U1 pad 32: CAN_RX -> LED_G
- U1 pad 33: CAN_TX -> LED_R
- U1 pad 35: GND -> Ext12
- U1 pad 36: Net-(U1-Pad36) -> USART3_RX
- U1 pad 38: Net-(U1-Pad38) -> +3V3
- U1 pad 39: /LCD_CLK -> Net-(U1-Pad39)
- U1 pad 4: Net-(U1-Pad4) -> /LCD_DIN
- U1 pad 8: Net-(U1-Pad8) -> CAN_RX
- U1 pad 9: Net-(U1-Pad9) -> CAN_TX
Routing:
- net GND: track 0.00 -> 311.1 mm, vias 0 -> 2
- net +3V3: track 0.00 -> 128.7 mm, vias 0 -> 2
- net SW_UP: track 0.00 -> 94.5 mm
- net LED_W: track 0.00 -> 70.9 mm, vias 0 -> 2
- net SW_LEFT: track 0.00 -> 66.1 mm
- net LED_R: track 0.00 -> 63.3 mm
- net LED_G: track 0.00 -> 61.0 mm, vias 0 -> 1
- net SW_DOWN: track 0.00 -> 57.4 mm
- net SW_RIGHT: track 0.00 -> 54.5 mm
- net LED_B: track 0.00 -> 53.3 mm, vias 0 -> 2
- net CAN_RX: track 0.00 -> 49.8 mm
- net OUT_W: track 0.00 -> 37.4 mm
- net CAN_TX: track 0.00 -> 37.1 mm
- net /Valt1: track 0.00 -> 32.9 mm
- net Net-(C1-Pad1): track 0.00 -> 31.9 mm
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
Commit message: PCB design
Parts:
- removed J5: Conn_01x04, Connector_PinHeader_2.54mm:PinHeader_1x04_P2.54mm_Vertical
- added J10: Conn_01x02, Connector_PinHeader_2.54mm:PinHeader_1x02_P2.54mm_Vertical, F.Cu at (76.2, 100.3)
- added J8: Conn_01x04, Connector_PinHeader_2.54mm:PinHeader_1x04_P2.54mm_Vertical, F.Cu at (76.2, 118.1)
- added J9: Conn_01x04, Connector_PinHeader_2.54mm:PinHeader_1x04_P2.54mm_Vertical, F.Cu at (138.4, 120.7)
- R1, R2, R3: footprint Resistor_THT:R_Axial_DIN0204_L3.6mm_D1.6mm_P7.62mm_Horizontal -> Resistor_THT:R_Axial_DIN0207_L6.3mm_D2.5mm_P15.24mm_Horizontal
- R4: footprint Resistor_THT:R_Axial_DIN0204_L3.6mm_D1.6mm_P7.62mm_Horizontal -> Resistor_THT:R_Axial_DIN0207_L6.3mm_D2.5mm_P10.16mm_Horizontal
- moved R5 78.0 mm to (200.7, 61.0)
- moved J4 73.3 mm to (204.5, 61.0)
- moved U4 69.4 mm to (189.2, 61.0)
- moved R6 52.2 mm to (111.8, 55.9)
- moved J15 46.7 mm to (81.3, 77.5), turned to 0 degrees
- moved U5 46.2 mm to (88.9, 100.3), turned to 180 degrees
- moved J11 46.2 mm to (156.2, 85.1)
- moved R3 45.2 mm to (143.5, 92.7)
- moved D1 44.2 mm to (88.9, 86.4)
- moved J2 44.2 mm to (81.3, 71.1)
- moved U1 44.2 mm to (108.0, 77.5)
- moved U2 44.2 mm to (95.2, 71.1)
- moved C1 42.7 mm to (86.7, 118.1), turned to 180 degrees
- moved SW1 42.4 mm to (154.9, 116.8), turned to 180 degrees
- moved J1 41.3 mm to (104.1, 94.0)
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Connections:
- net Ext2 renamed Net-(U1-Pad6)
- net Ext3 renamed Net-(U1-Pad7)
- net Ext4 renamed Net-(U1-Pad10)
- J11 pad 2: GND -> GND_SCL
- U1 pad 12: Ext5 -> SW_LEFT
- U1 pad 13: CAN_EN -> SW_UP
- U1 pad 14: Ext6 -> SW_RIGHT
- U1 pad 15: Ext7 -> SW_DOWN
- U1 pad 18: +5V -> Net-(J10-Pad1)
- U1 pad 19: GND -> GND_SCL
- U1 pad 22: SW_UP -> Net-(U1-Pad22)
- U1 pad 23: SW_DOWN -> Net-(U1-Pad23)
- U1 pad 24: SW_RIGHT -> Net-(U1-Pad24)
- U1 pad 25: SW_LEFT -> Net-(U1-Pad25)
- U1 pad 39: Net-(U1-Pad39) -> GND
- U1 pad 5: Ext1 -> CAN_EN
Routing:
- net Net-(J10-Pad1): track 0.00 -> 180.3 mm, vias 0 -> 2
- net +3V3: track 128.7 -> 233.1 mm, vias 2 -> 4
- net USART2_RX: track 0.00 -> 102.3 mm, vias 0 -> 2
- net USART2_TX: track 0.00 -> 97.2 mm, vias 0 -> 2
- net GND: track 311.1 -> 395.9 mm, vias 2 -> 9
- net USART3_RX: track 5.61 -> 71.2 mm
- net SW_UP: track 94.5 -> 39.0 mm
- net CAN_EN: track 0.00 -> 34.6 mm
- net SW_LEFT: track 66.1 -> 35.4 mm
- net OUT_R: track 0.00 -> 29.1 mm
- net LED_B: track 53.3 -> 80.5 mm, vias 2 -> 0
- net SW_RIGHT: track 54.5 -> 28.5 mm
- net +5V: track 9.80 -> 34.5 mm
- net LED_W: track 70.9 -> 47.4 mm, vias 2 -> 0
- net LED_R: track 63.3 -> 48.0 mm, vias 0 -> 2
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Other:
- board outline added: 137.2 x 74.9 mm
- net class Default: trace_width 0.25 -> 0.8; via_dia 0.8 -> 1.2
- rule trace_min: 0.2 -> 0.8

Commit message: update PCB
Parts:
- added J16: Conn_01x01, Connector_PinHeader_2.54mm:PinHeader_1x01_P2.54mm_Vertical, F.Cu at (119.4, 83.8)
- added J17: Conn_01x01, Connector_PinHeader_2.54mm:PinHeader_1x01_P2.54mm_Vertical, F.Cu at (123.2, 83.8)
- added J18: Conn_01x01, Connector_PinHeader_2.54mm:PinHeader_1x01_P2.54mm_Vertical, F.Cu at (127.0, 83.8)
- added J19: Conn_01x04, Connector_PinHeader_2.54mm:PinHeader_1x04_P2.54mm_Vertical, F.Cu at (146.1, 57.1)
- moved J1 3.81 mm to (104.1, 90.2)
Connections:
- U1 pad 10: Net-(U1-Pad10) -> TP3
- U1 pad 22: Net-(U1-Pad22) -> TP7
- U1 pad 23: Net-(U1-Pad23) -> TP6
- U1 pad 24: Net-(U1-Pad24) -> TP5
- U1 pad 25: Net-(U1-Pad25) -> TP4
- U1 pad 6: Net-(U1-Pad6) -> TP1
- U1 pad 7: Net-(U1-Pad7) -> TP2
Routing:
- net Net-(J10-Pad1): track 180.3 -> 3.81 mm, vias 2 -> 1
- net USART2_RX: track 102.3 -> 72.7 mm
- net +5V: track 34.5 -> 25.4 mm
- net GND: track 395.9 -> 388.7 mm
- net USART2_TX: track 97.2 -> 104.3 mm
- net SW_UP: track 39.0 -> 45.5 mm
- net TP7: track 0.00 -> 5.08 mm
- net /LCD_DIN: track 18.1 -> 14.3 mm
- net /LCD_CE: track 18.1 -> 14.3 mm
- net /LCD_DC: track 18.1 -> 14.3 mm
- net TP6: track 0.00 -> 3.81 mm
- net TP5: track 0.00 -> 3.81 mm
- net TP4: track 0.00 -> 3.81 mm
- net /LCD_RST: track 18.1 -> 14.3 mm
- net +3V3: track 233.1 -> 236.7 mm
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Other:
- net class Default: via_dia 1.2 -> 1.8; via_drill 0.4 -> 0.8

Commit message: update PCB
Parts:
- removed J17, J18: Conn_01x01, Connector_PinHeader_2.54mm:PinHeader_1x01_P2.54mm_Vertical
- added R11: R, Resistor_THT:R_Axial_DIN0207_L6.3mm_D2.5mm_P10.16mm_Horizontal, F.Cu at (119.4, 108.0)
- added R12: R, Resistor_THT:R_Axial_DIN0207_L6.3mm_D2.5mm_P10.16mm_Horizontal, F.Cu at (119.4, 113.0)
- C1: footprint Capacitor_SMD:CP_Elec_5x4.5 -> Capacitor_THT:CP_Radial_D6.3mm_P2.50mm
- C2: footprint Capacitor_SMD:CP_Elec_5x4.5 -> Capacitor_THT:CP_Radial_D5.0mm_P2.50mm
- J16: value Conn_01x01 -> Conn_01x03; footprint Connector_PinHeader_2.54mm:PinHeader_1x01_P2.54mm_Vertical -> Connector_PinHeader_2.54mm:PinHeader_1x03_P2.54mm_Vertical
- moved J14 24.1 mm to (104.1, 141.0)
- moved J12 19.3 mm to (172.7, 130.8)
- moved J13 19.3 mm to (190.5, 138.4)
- moved J3 19.3 mm to (199.4, 123.2)
- moved C1 18.1 mm to (96.5, 133.3)
- moved J16 15.5 mm to (128.3, 96.5), turned to 90 degrees
- moved J11 14.8 mm to (163.8, 97.8)
- moved J15 14.8 mm to (88.9, 90.2)
- moved J7 14.8 mm to (210.8, 85.1)
- moved R1 14.8 mm to (151.1, 109.2)
- moved R10 14.8 mm to (190.5, 95.2)
- moved R3 14.8 mm to (151.1, 105.4)
- moved R4 14.8 mm to (146.1, 113.0)
- moved R7 14.8 mm to (174.0, 102.9)
- moved R9 14.8 mm to (190.5, 90.2)
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Routing:
- net Net-(J10-Pad1): track 3.81 -> 130.9 mm, vias 1 -> 0
- net USART2_RX: track 72.7 -> 114.0 mm
- net GND: track 388.7 -> 421.6 mm
- net /LIGHT: track 0.00 -> 17.3 mm
- net +3V3: track 236.7 -> 225.3 mm
- net TP3: track 0.00 -> 9.94 mm
- net +5V: track 25.4 -> 34.9 mm
- net USART2_TX: track 104.3 -> 112.2 mm
- net /LCD_DIN: track 14.3 -> 21.2 mm
- net TP2: track 0.00 -> 6.35 mm
- net TP1: track 0.00 -> 6.35 mm
- net /LCD_CLK: track 30.3 -> 36.4 mm
- net /LCD_DC: track 14.3 -> 19.7 mm
- net /LCD_RST: track 14.3 -> 19.7 mm
- net /LCD_CE: track 14.3 -> 18.9 mm
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Other:
- board size 137.2 x 74.9 mm -> 137.2 x 81.3 mm
