File: PCB/stm_proto_board/stm_proto_board.sch (KiCad schematic (older format))
At the start: 38 parts, among them J1 Conn_01x08, J11 Conn_01x04, J12 Conn_01x04, J13 Conn_01x04, J14 Conn_01x08, J15 Conn_01x02, J2 Conn_01x04, J3 DB9_Female, J4 Conn_01x02, J5 Conn_01x04, J6 Conn_01x02, J7 Conn_01x04, SW1 SW_Push, SW2 SW_Push, SW3 SW_Push, SW4 SW_Push, U1 YAAJ_BluePill_Part_Like, U2 MCP2551-I-P, U3 MAX3232_convertor, U4 LTV-814, U5 L7805, U6 4N25, U7 4N25, U8 4N25, U9 4N25

Commit message: PCB design
Parts:
- added J10: Conn_01x02, Connector_PinHeader_2.54mm:PinHeader_1x02_P2.54mm_Vertical, symbol Connector_Generic:Conn_01x02
- added J8, J9: Conn_01x04, Connector_PinHeader_2.54mm:PinHeader_1x04_P2.54mm_Vertical, symbol Connector_Generic:Conn_01x04
- R1, R2, R3: footprint Resistor_THT:R_Axial_DIN0204_L3.6mm_D1.6mm_P7.62mm_Horizontal -> Resistor_THT:R_Axial_DIN0207_L6.3mm_D2.5mm_P15.24mm_Horizontal
- R4: footprint Resistor_THT:R_Axial_DIN0204_L3.6mm_D1.6mm_P7.62mm_Horizontal -> Resistor_THT:R_Axial_DIN0207_L6.3mm_D2.5mm_P10.16mm_Horizontal
Connections:
- net labels added: GND_SCL
- net labels removed: Ext1, Ext2, Ext3, Ext4, Ext5, Ext6, Ext7
- wire segments 185 -> 198
Changed lines of the file:
@@
-$EndComp
-$Comp
-L power:GND #PWR0102
-U 1 1 5B6EFA7C
-P 4500 5250
-F 0 "#PWR0102" H 4500 5000 50  0001 C CNN
-F 1 "GND" H 4505 5077 50  0000 C CNN
-F 2 "" H 4500 5250 50  0001 C CNN
-F 3 "" H 4500 5250 50  0001 C CNN
-	1    4500 5250
-	1    0    0    -1
 $EndComp
 $Comp
@@
 F 0 "R4" H 5870 7396 50  0000 L CNN
 F 1 "R" H 5870 7305 50  0000 L CNN
-F 2 "Resistor_THT:R_Axial_DIN0204_L3.6mm_D1.6mm_P7.62mm_Horizontal" V 5730 7350 50  0001 C CNN
+F 2 "Resistor_THT:R_Axial_DIN0207_L6.3mm_D2.5mm_P10.16mm_Horizontal" V 5730 7350 50  0001 C CNN
 F 3 "~" H 5800 7350 50  0001 C CNN
 	1    5800 7350
@@
 F 0 "R3" H 6120 7396 50  0000 L CNN
 F 1 "R" H 6120 7305 50  0000 L CNN
-F 2 "Resistor_THT:R_Axial_DIN0204_L3.6mm_D1.6mm_P7.62mm_Horizontal" V 5980 7350 50  0001 C CNN
+F 2 "Resistor_THT:R_Axial_DIN0207_L6.3mm_D2.5mm_P15.24mm_Horizontal" V 5980 7350 50  0001 C CNN
 F 3 "~" H 6050 7350 50  0001 C CNN
 	1    6050 7350
@@
 F 0 "R2" H 6370 7396 50  0000 L CNN
 F 1 "R" H 6370 7305 50  0000 L CNN
-F 2 "Resistor_THT:R_Axial_DIN0204_L3.6mm_D1.6mm_P7.62mm_Horizontal" V 6230 7350 50  0001 C CNN
+F 2 "Resistor_THT:R_Axial_DIN0207_L6.3mm_D2.5mm_P15.24mm_Horizontal" V 6230 7350 50  0001 C CNN
 F 3 "~" H 6300 7350 50  0001 C CNN
 	1    6300 7350
@@
 F 0 "R1" H 6620 7396 50  0000 L CNN
 F 1 "R" H 6620 7305 50  0000 L CNN
-F 2 "Resistor_THT:R_Axial_DIN0204_L3.6mm_D1.6mm_P7.62mm_Horizontal" V 6480 7350 50  0001 C CNN
+F 2 "Resistor_THT:R_Axial_DIN0207_L6.3mm_D2.5mm_P15.24mm_Horizontal" V 6480 7350 50  0001 C CNN
 F 3 "~" H 6550 7350 50  0001 C CNN
 	1    6550 7350
@@
 Wire Wire Line
 	5500 6750 5600 6750
-Text GLabel 6700 5000 2    50   Input ~ 0
+Text GLabel 4800 4400 0    50   Input ~ 0
 SW_UP
 Text GLabel 5700 6250 2    50   Output ~ 0
@@
 	4950 4000 4800 4000
 Wire Wire Line
-	4500 5000 4500 5250
-Wire Wire Line
 	6750 3400 6750 3250
 Wire Wire Line
@@
 Wire Wire Line
 	6550 3600 6650 3600
-Text GLabel 4800 4400 0    50   Output ~ 0
+Text GLabel 4750 3600 0    50   Output ~ 0
 CAN_EN
 Wire Wire Line
-	4950 4400 4800 4400
+	4950 4600 4800 4600
 Wire Wire Line
 	10150 3450 9950 3450
@@
 Wire Wire Line
 	4950 4700 4850 4700
-Text GLabel 6700 4900 2    50   Input ~ 0
+Text GLabel 4800 4600 0    50   Input ~ 0
 SW_DOWN
-Text GLabel 6700 4800 2    50   Input ~ 0
+Text GLabel 4800 4500 0    50   Input ~ 0
 SW_RIGHT
-Text GLabel 6700 4700 2    50   Input ~ 0
+Text GLabel 4800 4300 0    50   Input ~ 0
 SW_LEFT
 Wire Wire Line
@@
 L power:+5V #PWR0119
 U 1 1 5B8AAD24
-P 4500 4900
-F 0 "#PWR0119" H 4500 4750 50  0001 C CNN
-F 1 "+5V" H 4515 5073 50  0000 C CNN
-F 2 "" H 4500 4900 50  0001 C CNN
-F 3 "" H 4500 4900 50  0001 C CNN
-	1    4500 4900
+P 4450 5450
+F 0 "#PWR0119" H 4450 5300 50  0001 C CNN
+F 1 "+5V" H 4465 5623 50  0000 C CNN
+F 2 "" H 4450 5450 50  0001 C CNN
+F 3 "" H 4450 5450 50  0001 C CNN
+	1    4450 5450
 	1    0    0    -1
 $EndComp
@@
 	1    0    0    -1
 $EndComp
-$Comp
-L power:GND #PWR0127
-U 1 1 5BE0BBDC
-P 6000 2200
-F 0 "#PWR0127" H 6000 1950 50  0001 C CNN
-F 1 "GND" H 6005 2027 50  0000 C CNN
-F 2 "" H 6000 2200 50  0001 C CNN
-F 3 "" H 6000 2200 50  0001 C CNN
-	1    6000 2200
-	1    0    0    -1
-$EndComp
 Text GLabel 6400 2100 0    50   BiDi ~ 0
 SDA
@@
 Wire Wire Line
 	6500 1900 6350 1900
-Wire Wire Line
-	6000 2000 6000 2200
-Wire Wire Line
-	6000 2000 6500 2000
 Wire Wire Line
 	6500 2100 6400 2100
@@
 Wire Wire Line
 	6550 4100 6650 4100
-Text GLabel 4750 3600 0    50   Input ~ 0
-Ext1
-Text GLabel 4750 3700 0    50   Input ~ 0
-Ext2
-Text GLabel 4750 3800 0    50   Input ~ 0
-Ext3
-Text GLabel 4750 4300 0    50   Input ~ 0
-Ext5
-Text GLabel 4750 4500 0    50   Input ~ 0
-Ext6
-Text GLabel 4750 4600 0    50   Input ~ 0
-Ext7
 Text GLabel 6700 3700 2    50   Input ~ 0
 Ext12
@@
 	4300 600  4300 2500
 Wire Wire Line
-	4500 4900 4950 4900
-Wire Wire Line
 	6700 4600 6550 4600
 Wire Wire Line
@@
 	4750 3800 4950 3800
 Wire Wire Line
-	4950 4300 4750 4300
-Wire Wire Line
-	4750 4500 4950 4500
-Wire Wire Line
-	4950 4600 4750 4600
-Text GLabel 4750 4100 0    50   Input ~ 0
-Ext4
-Wire Wire Line
 	4750 4100 4950 4100
-Wire Wire Line
-	4500 5000 4950 5000
 $Comp
 L power:+3V3 #PWR0132
 U 1 1 5FA7F8AA
-P 4700 5250
-F 0 "#PWR0132" H 4700 5100 50  0001 C CNN
-F 1 "+3V3" H 4715 5423 50  0000 C CNN
-F 2 "" H 4700 5250 50  0001 C CNN
-F 3 "" H 4700 5250 50  0001 C CNN
-	1    4700 5250
-	1    0    0    -1
+P 4950 5350
+F 0 "#PWR0132" H 4950 5200 50  0001 C CNN
+F 1 "+3V3" H 4965 5523 50  0000 C CNN
+F 2 "" H 4950 5350 50  0001 C CNN
+F 3 "" H 4950 5350 50  0001 C CNN
+	1    4950 5350
+	0    1    1    0
 $EndComp
 Wire Wire Line
 	4950 5100 4900 5100
-Wire Wire Line
-	4900 5100 4900 5250
-Wire Wire Line
-	4900 5250 4700 5250
 Wire Bus Line
 	900  5350 4300 5350
@@
 Wire Notes Line
 	4300 7500 800  7500
-Wire Notes Line
-	800  6000 4300 6000
 Connection ~ 3750 6450
 Wire Wire Line
@@
 	1    0    0    -1
 $EndComp
-Wire Notes Line
-	4300 6000 4300 7500
 Text Notes 4000 7400 0    50   ~ 0
 Power
@@
 Valt1
 Wire Wire Line
-	3750 7000 3750 7100
+	3750 7000 3750 7050
 Wire Wire Line
 	2550 7000 2550 7150
@@
 Wire Notes Line
 	2000 5100 4150 5100
+Wire Wire Line
+	4950 4400 4800 4400
+Wire Wire Line
+	4800 4500 4950 4500
+Wire Wire Line
+	4800 4300 4950 4300
+$Comp
+L Connector_Generic:Conn_01x04 J9
+U 1 1 5FB0D931
+P 4150 7050
+F 0 "J9" H 4230 7042 50  0000 L CNN
+F 1 "Conn_01x04" H 4230 6951 50  0000 L CNN
+F 2 "Connector_PinHeader_2.54mm:PinHeader_1x04_P2.54mm_Vertical" H 4150 7050 50  0001 C CNN
+F 3 "~" H 4150 7050 50  0001 C CNN
+	1    4150 7050
+	1    0    0    -1
+$EndComp
+Wire Wire Line
+	3750 6450 3950 6450
+Connection ~ 3950 6450
+Wire Wire Line
+	3950 7250 3950 7150
+Connection ~ 3950 7050
+Wire Wire Line
+	3950 7050 3950 6950
+Connection ~ 3950 7150
+Wire Wire Line
+	3950 7150 3950 7050
+Wire Wire Line
+	3750 7050 3950 7050
+Connection ~ 3750 7050
+Wire Wire Line
+	3750 7050 3750 7100
+Wire Wire Line
+	3950 6350 3950 6450
+Wire Wire Line
+	3950 6250 3950 6350
+Connection ~ 3950 6350
+$Comp
+L Connector_Generic:Conn_01x04 J8
+U 1 1 5FB00AF7
+P 4150 6350
+F 0 "J8" H 4230 6342 50  0000 L CNN
+F 1 "Conn_01x04" H 4230 6251 50  0000 L CNN
+F 2 "Connector_PinHeader_2.54mm:PinHeader_1x04_P2.54mm_Vertical" H 4150 6350 50  0001 C CNN
+F 3 "~" H 4150 6350 50  0001 C CNN
+	1    4150 6350
+	1    0    0    -1
+$EndComp
+Wire Wire Line
+	3950 6450 3950 6550
+$Comp
+L Connector_Generic:Conn_01x02 J10
+U 1 1 5FBF46C0
+P 4150 5650
+F 0 "J10" H 4230 5642 50  0000 L CNN
+F 1 "Conn_01x02" H 4230 5551 50  0000 L CNN
+F 2 "Connector_PinHeader_2.54mm:PinHeader_1x02_P2.54mm_Vertical" H 4150 5650 50  0001 C CNN
+F 3 "~" H 4150 5650 50  0001 C CNN
+	1    4150 5650
+	-1   0    0    1
+$EndComp
+Wire Wire Line
+	4900 5100 4900 5350
+Wire Wire Line
+	4900 5350 4950 5350
+Wire Wire Line
+	4350 5550 4450 5550
+Wire Notes Line
+	4300 6000 4300 7500
+Wire Notes Line
+	800  6000 4300 6000
+Wire Wire Line
+	4450 5550 4450 5450
+Wire Wire Line
+	4350 5650 4600 5650
+Wire Wire Line
+	4600 5650 4600 4900
+Wire Wire Line
+	4600 4900 4950 4900
+$Comp
+L power:GND #PWR0102
+U 1 1 5B6EFA7C
+P 6550 3000
+F 0 "#PWR0102" H 6550 2750 50  0001 C CNN
+F 1 "GND" H 6555 2827 50  0000 C CNN
+F 2 "" H 6550 3000 50  0001 C CNN
+F 3 "" H 6550 3000 50  0001 C CNN
+	1    6550 3000
+	-1   0    0    1
+$EndComp
+Wire Wire Line
+	6550 3000 6550 3200
+Text GLabel 6400 2000 0    50   Input ~ 0
+GND_SCL
+Wire Wire Line
+	6400 2000 6500 2000
+Text GLabel 4800 5100 3    50   Input ~ 0
+GND_SCL
+Wire Wire Line
+	4950 5000 4800 5000
+Wire Wire Line
+	4800 5000 4800 5100
 Wire Bus Line
 	4300 3300 4300 5350

Commit message: update PCB
Parts:
- added J16, J17, J18: Conn_01x01, Connector_PinHeader_2.54mm:PinHeader_1x01_P2.54mm_Vertical, symbol Connector_Generic:Conn_01x01
- added J19: Conn_01x04, Connector_PinHeader_2.54mm:PinHeader_1x04_P2.54mm_Vertical, symbol Connector_Generic:Conn_01x04
Connections:
- net labels added: TP1, TP2, TP3, TP4, TP5, TP6, TP7
Other:
- moved on the sheet: J15, J2, U2
Changed lines of the file:
@@
 L Interface_CAN_LIN:MCP2551-I-P U2
 U 1 1 5B6EF31C
-P 8800 1650
-F 0 "U2" H 8800 2228 50  0000 C CNN
-F 1 "MCP2551-I-P" H 8800 2137 50  0000 C CNN
-F 2 "Package_DIP:DIP-8_W7.62mm" H 8800 1150 50  0001 C CIN
-F 3 "http://ww1.microchip.com/downloads/en/devicedoc/21667d.pdf" H 8800 1650 50  0001 C CNN
-	1    8800 1650
+P 8850 1550
+F 0 "U2" H 8850 2128 50  0000 C CNN
+F 1 "MCP2551-I-P" H 8850 2037 50  0000 C CNN
+F 2 "Package_DIP:DIP-8_W7.62mm" H 8850 1050 50  0001 C CIN
+F 3 "http://ww1.microchip.com/downloads/en/devicedoc/21667d.pdf" H 8850 1550 50  0001 C CNN
+	1    8850 1550
 	1    0    0    -1
 $EndComp
@@
 L Connector_Generic:Conn_01x04 J2
 U 1 1 5B6EF715
-P 10000 1550
-F 0 "J2" H 10080 1542 50  0000 L CNN
-F 1 "Conn_01x04" H 10080 1451 50  0000 L CNN
-F 2 "Connector_PinHeader_2.54mm:PinHeader_1x04_P2.54mm_Horizontal" H 10000 1550 50  0001 C CNN
-F 3 "~" H 10000 1550 50  0001 C CNN
-	1    10000 1550
+P 10050 1450
+F 0 "J2" H 10130 1442 50  0000 L CNN
+F 1 "Conn_01x04" H 10130 1351 50  0000 L CNN
+F 2 "Connector_PinHeader_2.54mm:PinHeader_1x04_P2.54mm_Horizontal" H 10050 1450 50  0001 C CNN
+F 3 "~" H 10050 1450 50  0001 C CNN
+	1    10050 1450
 	1    0    0    -1
 $EndComp
@@
 L power:+3.3V #PWR0105
 U 1 1 5B6EE504
-P 8800 1050
-F 0 "#PWR0105" H 8800 900 50  0001 C CNN
-F 1 "+3.3V" H 8815 1223 50  0000 C CNN
-F 2 "" H 8800 1050 50  0001 C CNN
-F 3 "" H 8800 1050 50  0001 C CNN
-	1    8800 1050
-	1    0    0    -1
-$EndComp
-Wire Wire Line
-	8800 1250 8800 1050
+P 8850 950
+F 0 "#PWR0105" H 8850 800 50  0001 C CNN
+F 1 "+3.3V" H 8865 1123 50  0000 C CNN
+F 2 "" H 8850 950 50  0001 C CNN
+F 3 "" H 8850 950 50  0001 C CNN
+	1    8850 950
+	1    0    0    -1
+$EndComp
+Wire Wire Line
+	8850 1150 8850 950
 $Comp
 L power:GND #PWR0106
 U 1 1 5B6EE5EC
-P 8800 2200
-F 0 "#PWR0106" H 8800 1950 50  0001 C CNN
-F 1 "GND" H 8805 2027 50  0000 C CNN
-F 2 "" H 8800 2200 50  0001 C CNN
-F 3 "" H 8800 2200 50  0001 C CNN
-	1    8800 2200
-	1    0    0    -1
-$EndComp
-Wire Wire Line
-	8800 2050 8800 2200
-Wire Wire Line
-	9800 1550 9300 1550
-Wire Wire Line
-	9300 1750 9450 1750
-Wire Wire Line
-	9450 1750 9450 1650
-Wire Wire Line
-	9450 1650 9800 1650
-Text Label 9550 1450 0    50   ~ 0
+P 8850 2100
+F 0 "#PWR0106" H 8850 1850 50  0001 C CNN
+F 1 "GND" H 8855 1927 50  0000 C CNN
+F 2 "" H 8850 2100 50  0001 C CNN
+F 3 "" H 8850 2100 50  0001 C CNN
+	1    8850 2100
+	1    0    0    -1
+$EndComp
+Wire Wire Line
+	8850 1950 8850 2100
+Wire Wire Line
+	9850 1450 9350 1450
+Wire Wire Line
+	9350 1650 9500 1650
+Wire Wire Line
+	9500 1650 9500 1550
+Wire Wire Line
+	9500 1550 9850 1550
+Text Label 9600 1350 0    50   ~ 0
 Valt1
 Wire Wire Line
-	9550 1450 9800 1450
-Text Label 9550 1750 0    50   ~ 0
+	9600 1350 9850 1350
+Text Label 9600 1650 0    50   ~ 0
 Valt2
 Wire Wire Line
-	9550 1750 9800 1750
-Text Label 2050 4250 0    50   ~ 0
+	9600 1650 9850 1650
+Text Label 1750 4250 0    50   ~ 0
 LCD_RST
-Text Label 2050 4350 0    50   ~ 0
+Text Label 1750 4350 0    50   ~ 0
 LCD_CE
-Text Label 2050 4450 0    50   ~ 0
+Text Label 1750 4450 0    50   ~ 0
 LCD_DC
-Text Label 2050 4550 0    50   ~ 0
+Text Label 1750 4550 0    50   ~ 0
 LCD_DIN
-Text Label 2050 4650 0    50   ~ 0
+Text Label 1750 4650 0    50   ~ 0
 LCD_CLK
-Text Label 2150 4750 0    50   ~ 0
+Text Label 1850 4750 0    50   ~ 0
 VCC
-Text Label 2100 4850 0    50   ~ 0
+Text Label 1800 4850 0    50   ~ 0
 LIGHT
-Text Label 2150 4950 0    50   ~ 0
+Text Label 1900 4950 0    50   ~ 0
 GND
 $Comp
@@
 Wire Wire Line
 	1300 4750 2350 4750
-Text GLabel 8150 1450 0    50   Input ~ 0
+Text GLabel 8200 1350 0    50   Input ~ 0
 CAN_TX
-Text GLabel 8150 1550 0    50   Input ~ 0
+Text GLabel 8200 1450 0    50   Input ~ 0
 CAN_RX
-Text GLabel 8150 1850 0    50   Input ~ 0
+Text GLabel 8200 1750 0    50   Input ~ 0
 CAN_EN
 Wire Wire Line
-	8300 1450 8150 1450
-Wire Wire Line
-	8300 1550 8150 1550
-Wire Wire Line
-	8150 1850 8300 1850
+	8350 1350 8200 1350
+Wire Wire Line
+	8350 1450 8200 1450
+Wire Wire Line
+	8200 1750 8350 1750
 Entry Wire Line
 	1000 4450 900  4550
@@
 EDF Teleinfo
 Wire Notes Line
-	7600 2500 10700 2500
-Wire Notes Line
-	10700 2500 10700 800
-Wire Notes Line
-	10700 800  7600 800
-Wire Notes Line
-	7600 800  7600 2500
-Text Notes 10200 2400 0    50   ~ 0
+	7650 2400 10750 2400
+Wire Notes Line
+	10750 2400 10750 700
+Wire Notes Line
+	10750 700  7650 700
+Wire Notes Line
+	7650 700  7650 2400
+Text Notes 10250 2300 0    50   ~ 0
 CAN Link
 Wire Notes Line
-	2000 4100 2000 5100
+	2300 4100 2300 5100
 Wire Notes Line
 	4150 5100 4150 4100
@@
 Wire Wire Line
 	6550 4200 6650 4200
-Text Label 9550 1100 0    50   ~ 0
+Text Label 9600 1000 0    50   ~ 0
 Valt1
 Wire Wire Line
-	9550 1100 9800 1100
-Text Label 9550 1200 0    50   ~ 0
+	9600 1000 9850 1000
+Text Label 9600 1100 0    50   ~ 0
 Valt2
 Wire Wire Line
-	9550 1200 9800 1200
+	9600 1100 9850 1100
 $Comp
 L Connector_Generic:Conn_01x02 J15
 U 1 1 603342BF
-P 10000 1100
-F 0 "J15" H 10080 1092 50  0000 L CNN
-F 1 "Conn_01x02" H 10080 1001 50  0000 L CNN
-F 2 "Connector_PinHeader_2.54mm:PinHeader_1x02_P2.54mm_Vertical" H 10000 1100 50  0001 C CNN
-F 3 "~" H 10000 1100 50  0001 C CNN
-	1    10000 1100
+P 10050 1000
+F 0 "J15" H 10130 992 50  0000 L CNN
+F 1 "Conn_01x02" H 10130 901 50  0000 L CNN
+F 2 "Connector_PinHeader_2.54mm:PinHeader_1x02_P2.54mm_Vertical" H 10050 1000 50  0001 C CNN
+F 3 "~" H 10050 1000 50  0001 C CNN
+	1    10050 1000
 	1    0    0    -1
 $EndComp
@@
 	1    0    0    -1
 $EndComp
-Wire Notes Line
-	2000 4100 4150 4100
-Wire Notes Line
-	2000 5100 4150 5100
 Wire Wire Line
 	4950 4400 4800 4400
@@
 Wire Wire Line
 	4800 5000 4800 5100
+$Comp
+L Connector_Generic:Conn_01x01 J16
+U 1 1 5F91D967
+P 4950 800
+F 0 "J16" H 5030 842 50  0000 L CNN
+F 1 "Conn_01x01" H 5030 751 50  0000 L CNN
+F 2 "Connector_PinHeader_2.54mm:PinHeader_1x01_P2.54mm_Vertical" H 4950 800 50  0001 C CNN
+F 3 "~" H 4950 800 50  0001 C CNN
+	1    4950 800
+	1    0    0    -1
+$EndComp
+$Comp
+L Connector_Generic:Conn_01x01 J17
+U 1 1 5F924708
+P 4950 1000
+F 0 "J17" H 5030 1042 50  0000 L CNN
+F 1 "Conn_01x01" H 5030 951 50  0000 L CNN
+F 2 "Connector_PinHeader_2.54mm:PinHeader_1x01_P2.54mm_Vertical" H 4950 1000 50  0001 C CNN
+F 3 "~" H 4950 1000 50  0001 C CNN
+	1    4950 1000
+	1    0    0    -1
+$EndComp
+$Comp
+L Connector_Generic:Conn_01x01 J18
+U 1 1 5F932C0D
+P 4950 1200
+F 0 "J18" H 5030 1242 50  0000 L CNN
+F 1 "Conn_01x01" H 5030 1151 50  0000 L CNN
+F 2 "Connector_PinHeader_2.54mm:PinHeader_1x01_P2.54mm_Vertical" H 4950 1200 50  0001 C CNN
+F 3 "~" H 4950 1200 50  0001 C CNN
+	1    4950 1200
+	1    0    0    -1
+$EndComp
+Text GLabel 4750 800  0    50   Input ~ 0
+TP1
+Text GLabel 4750 1000 0    50   Input ~ 0
+TP2
+Text GLabel 4750 1200 0    50   Input ~ 0
+TP3
+Text GLabel 4750 1400 0    50   Input ~ 0
+TP4
+Text GLabel 4750 3700 0    50   Input ~ 0
+TP1
+Text GLabel 4750 3800 0    50   Input ~ 0
+TP2
+Text GLabel 4750 4100 0    50   Input ~ 0
+TP3
+Text GLabel 4750 1500 0    50   Input ~ 0
+TP5
+Text GLabel 4750 1600 0    50   Input ~ 0
+TP6
+Text GLabel 6700 4700 2    50   Input ~ 0
+TP4
+Text GLabel 6700 4800 2    50   Input ~ 0
+TP5
+Text GLabel 6700 4900 2    50   Input ~ 0
+TP6
+Text GLabel 4750 1700 0    50   Input ~ 0
+TP7
+Text GLabel 6700 5000 2    50   Input ~ 0
+TP7
+$Comp
+L Connector_Generic:Conn_01x04 J19
+U 1 1 5FBFD4E3
+P 4950 1500
+F 0 "J19" H 5030 1492 50  0000 L CNN
+F 1 "Conn_01x04" H 5030 1401 50  0000 L CNN
+F 2 "Connector_PinHeader_2.54mm:PinHeader_1x04_P2.54mm_Vertical" H 4950 1500 50  0001 C CNN
+F 3 "~" H 4950 1500 50  0001 C CNN
+	1    4950 1500
+	1    0    0    -1
+$EndComp
+Wire Notes Line
+	4150 4100 2300 4100
+Wire Notes Line
+	4150 5100 2300 5100
 Wire Bus Line
 	4300 3300 4300 5350
