File: PCB/raspberrypi_shield/raspberrypi_shield.kicad_pcb (KiCad board)
At the start: 2 copper layers, 49 parts, among them J1 Conn_01x03, J10 Conn_01x02, J11 Conn_01x07, J12 Conn_02x20_Odd_Even, J13 Conn_01x04, J14 Conn_01x04, J15 Conn_01x04, J2 Conn_01x03, J3 Conn_01x03, J4 Conn_01x03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

Commit message: Update schematic
Parts:
- moved J10 194.4 mm to (268.0, 104.1), turned to 270 degrees
- moved U6 187.6 mm to (265.4, 99.1), turned to 90 degrees
- moved J8 182.3 mm to (257.8, 104.1), turned to 270 degrees
- moved R10 180.2 mm to (268.0, 82.5), turned to 270 degrees
- moved U4 175.4 mm to (255.3, 99.1), turned to 90 degrees
- moved J9 170.6 mm to (247.7, 104.1), turned to 270 degrees
- moved R8 167.1 mm to (257.8, 82.5), turned to 270 degrees
- moved U5 163.5 mm to (245.1, 99.1), turned to 90 degrees
- moved J7 159.4 mm to (237.5, 104.1), turned to 270 degrees
- moved D1 158.8 mm to (214.6, 83.8)
- moved D2 158.8 mm to (214.6, 66.0)
- moved D3 158.8 mm to (214.6, 48.3)
- moved D4 158.8 mm to (214.6, 30.5)
- moved J1 158.8 mm to (188.0, 82.5)
- moved J2 158.8 mm to (188.0, 64.8)
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