File: PCB/raspberrypi_shield/raspberrypi_shield.sch (KiCad schematic (older format))
At the start: 54 parts, among them J1 Conn_01x03, J10 Conn_01x02, J11 Conn_01x07, J12 Conn_02x20_Odd_Even, J13 Conn_01x04, J14 Conn_01x04, J15 Conn_01x04, J2 Conn_01x03, J3 Conn_01x03, J4 Conn_01x03, J5 Conn_01x02, J6 Conn_01x02, J7 Conn_01x02, J8 Conn_01x02, J9 Conn_01x02, K1 SANYOU_SRD_Form_C, K2 SANYOU_SRD_Form_C, K3 SANYOU_SRD_Form_C, K4 SANYOU_SRD_Form_C, Q1 2N2219, Q2 2N2219, Q3 2N2219, Q4 2N2219, U1 MCP2515-xSO, U2 MCP2551-I-P, U3 4N25, U4 4N25, U5 4N25, U6 4N25, U7 DHT11, Y1 8M

Commit message: Update schematic
Connections:
- net labels added: Relay2, Relay3, Relay4
Changed lines of the file:
@@
 	1800 4800 2250 4800
 Text GLabel 1000 4950 0    50   Input ~ 0
-Relay1
+Relay2
 Wire Wire Line
 	1550 5250 1800 5250
@@
 	1800 5700 2250 5700
 Text GLabel 1000 5850 0    50   Input ~ 0
-Relay1
+Relay3
 Wire Wire Line
 	1550 6150 1800 6150
@@
 	1800 6650 2250 6650
 Text GLabel 1000 6800 0    50   Input ~ 0
-Relay1
+Relay4
 Wire Wire Line
 	1550 7100 1800 7100
@@
 Wire Wire Line
 	2650 750  2650 1000
-Text GLabel 10650 3100 2    50   Input ~ 0
+Text GLabel 10500 2700 2    50   Input ~ 0
 Input1
-Text GLabel 10650 3200 2    50   Input ~ 0
+Text GLabel 10500 2800 2    50   Input ~ 0
 Input2
-Text GLabel 10650 3300 2    50   Input ~ 0
+Text GLabel 10500 2900 2    50   Input ~ 0
 Input3
-Text GLabel 10650 3400 2    50   Input ~ 0
+Text GLabel 10500 3000 2    50   Input ~ 0
 Input3
 $Comp
@@
 Wire Wire Line
 	8800 1300 9350 1300
+Text GLabel 8850 2400 0    50   Input ~ 0
+Relay1
+Text GLabel 8850 2500 0    50   Input ~ 0
+Relay2
+Text GLabel 8850 2600 0    50   Input ~ 0
+Relay3
+Text GLabel 8850 2700 0    50   Input ~ 0
+Relay4
 $EndSCHEMATC

Commit message: update schematics
Parts:
- added BZ?: Buzzer, symbol Device:Buzzer
- added R?: R, symbol Device:R
Connections:
- net labels added: buzz
- wire segments 230 -> 231
Changed lines of the file:
@@
 Wire Wire Line
 	8800 1300 9350 1300
-Text GLabel 8850 2400 0    50   Input ~ 0
+Text GLabel 8850 2400 0    50   Output ~ 0
 Relay1
-Text GLabel 8850 2500 0    50   Input ~ 0
+Text GLabel 8850 2500 0    50   Output ~ 0
 Relay2
-Text GLabel 8850 2600 0    50   Input ~ 0
+Text GLabel 8850 2600 0    50   Output ~ 0
 Relay3
-Text GLabel 8850 2700 0    50   Input ~ 0
+Text GLabel 8850 2700 0    50   Output ~ 0
 Relay4
+$Comp
+L Device:Buzzer BZ?
+U 1 1 5FA86580
+P 5850 6250
+F 0 "BZ?" H 6002 6279 50  0000 L CNN
+F 1 "Buzzer" H 6002 6188 50  0000 L CNN
+F 2 "" V 5825 6350 50  0001 C CNN
+F 3 "~" V 5825 6350 50  0001 C CNN
+	1    5850 6250
+	1    0    0    -1
+$EndComp
+$Comp
+L Device:R R?
+U 1 1 5FA99F14
+P 5550 6150
+F 0 "R?" V 5343 6150 50  0000 C CNN
+F 1 "R" V 5434 6150 50  0000 C CNN
+F 2 "" V 5480 6150 50  0001 C CNN
+F 3 "~" H 5550 6150 50  0001 C CNN
+	1    5550 6150
+	0    1    1    0
+$EndComp
+Wire Wire Line
+	5750 6150 5700 6150
+$Comp
+L power:GND #PWR?
+U 1 1 5FB10533
+P 5750 6350
+F 0 "#PWR?" H 5750 6100 50  0001 C CNN
+F 1 "GND" H 5755 6177 50  0000 C CNN
+F 2 "" H 5750 6350 50  0001 C CNN
+F 3 "" H 5750 6350 50  0001 C CNN
+	1    5750 6350
+	1    0    0    -1
+$EndComp
+Text GLabel 5400 6150 0    50   Input ~ 0
+buzz
+Text GLabel 8850 2800 0    50   Output ~ 0
+buzz
 $EndSCHEMATC
