File: PCB/stm_intercom_door_entrance/stm_intercom_door_entrance.kicad_pcb (KiCad board)
At the start: 2 copper layers, 47 parts, among them J1 Conn_01x02, J10 Conn_01x02, J11 Conn_01x04, J12 Conn_01x04, J13 Conn_01x04, J14 Conn_01x02, J15 Conn_01x02, J16 Conn_01x01, J17 Conn_01x03, J18 Conn_01x03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

Commit message: Update schematic
Parts:
- added J20: Conn_01x08, Connector_PinHeader_2.54mm:PinHeader_1x08_P2.54mm_Vertical, F.Cu at (162.6, 161.3)
- D2, D3: footprint Diode_THT:Diode_Bridge_DIP-4_W7.62mm_P5.08mm -> Diode_THT:D_5W_P10.16mm_Horizontal
- moved J5 132.9 mm to (108.0, 176.5), turned to 180 degrees
- moved J11 115.1 mm to (100.3, 176.5), turned to 180 degrees
- moved J12 103.2 mm to (247.7, 170.2), turned to 180 degrees
- moved J1 50.1 mm to (248.3, 110.4)
- moved J10 50.1 mm to (239.0, 110.9)
- moved J19 50.1 mm to (234.3, 110.9)
- moved J7 50.1 mm to (243.6, 110.9)
- moved C3 50.1 mm to (245.4, 119.1)
- moved C5 50.1 mm to (238.7, 119.1)
- moved J3 32.7 mm to (237.5, 133.3)
Connections:
- net +3V3 renamed VCC
- net IRQ renamed I2C_IRQ
- net SCL renamed I2C_SCL
- net SDA renamed I2C_SDA
- J11 pad 2: GND_SCL -> GND
- U1 pad 30: Net-(U1-Pad30) -> PN_SCK
- U1 pad 31: Net-(U1-Pad31) -> PN_MISO
- U1 pad 32: Net-(U1-Pad32) -> PN_MOSI
- U1 pad 33: Net-(U1-Pad33) -> PN_SS
- U1 pad 34: Net-(U1-Pad34) -> PN_IRQ
- U1 pad 35: Net-(U1-Pad35) -> PN_RSTO

Commit message: update schematics
Parts:
- added BZ1: Buzzer, Buzzer_Beeper:Buzzer_12x9.5RM7.6, F.Cu at (161.0, 108.5)
- added J21: Conn_01x04, Connector_PinHeader_2.54mm:PinHeader_1x04_P2.54mm_Vertical, F.Cu at (212.0, 99.5)
- added J23: Conn_01x02, Connector_PinHeader_2.54mm:PinHeader_1x02_P2.54mm_Vertical, F.Cu at (150.5, 126.5)
- added J24: Conn_01x02, Connector_PinHeader_2.54mm:PinHeader_1x02_P2.54mm_Vertical, F.Cu at (151.0, 146.5)
- added R10: R, Resistor_THT:R_Axial_DIN0204_L3.6mm_D1.6mm_P7.62mm_Horizontal, F.Cu at (161.0, 103.5)
- added R11: 330, Resistor_THT:R_Axial_DIN0204_L3.6mm_D1.6mm_P5.08mm_Vertical, F.Cu at (152.0, 130.5)
- added R12: 330, Resistor_THT:R_Axial_DIN0204_L3.6mm_D1.6mm_P5.08mm_Vertical, F.Cu at (152.0, 133.0)
- added R13: 330, Resistor_THT:R_Axial_DIN0204_L3.6mm_D1.6mm_P5.08mm_Vertical, F.Cu at (152.1, 142.5)
- J3: footprint Connector_PinHeader_2.54mm:PinHeader_1x04_P2.54mm_Horizontal -> Connector_PinHeader_2.54mm:PinHeader_1x04_P2.54mm_Vertical
- moved J6 141.8 mm to (85.5, 144.5)
- moved C5 132.5 mm to (107.5, 137.5), turned to 90 degrees
- moved J15 130.6 mm to (89.5, 110.5)
- moved U4 129.9 mm to (93.5, 131.0)
- moved J4 127.9 mm to (85.5, 133.0)
- moved J10 124.0 mm to (115.0, 111.5), turned to 180 degrees
- moved J12 122.6 mm to (125.5, 159.5)
- moved R7 121.0 mm to (93.5, 139.5)
- moved C6 115.7 mm to (107.5, 148.5), turned to 90 degrees
- moved C2 113.4 mm to (108.5, 123.0), turned to 180 degrees
- moved D1 108.9 mm to (101.0, 114.5), turned to 180 degrees
- moved R3 107.7 mm to (89.5, 140.5), turned to 270 degrees
- moved C1 107.0 mm to (98.0, 122.0), turned to 180 degrees
- moved Q1 105.4 mm to (156.5, 128.0)
- moved D2 104.3 mm to (168.0, 123.0)
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Connections:
- net Net-(J2-Pad2) renamed /CANH
- net Net-(J2-Pad3) renamed /CANL
- U1 pad 22: Net-(U1-Pad22) -> led3
- U1 pad 25: Net-(U1-Pad25) -> led2
- U1 pad 26: Net-(U1-Pad26) -> led1
- U1 pad 29: Net-(U1-Pad29) -> PN_RSTO
- U1 pad 35: PN_RSTO -> Net-(U1-Pad35)
- U1 pad 4: Net-(U1-Pad4) -> buzz
- U1 pad 6: USART2_TX -> USART1_TX
- U1 pad 7: USART2_RX -> USART1_RX
Routing:
- net VCC: track 0.00 -> 153.2 mm
- net GND: track 0.00 -> 56.9 mm
- net door_bell_2: track 0.00 -> 50.0 mm
- net USART2_RX: track 0.00 -> 46.0 mm
- net I2C_SCL: track 0.00 -> 44.3 mm
- net door_bell_1: track 0.00 -> 43.1 mm
- net I2C_SDA: track 0.00 -> 39.9 mm
- net USART2_TX: track 0.00 -> 36.2 mm
- net Net-(J10-Pad1): track 0.00 -> 34.9 mm, vias 0 -> 2
- net /Valt2: track 0.00 -> 33.9 mm
- net PN_RSTO: track 0.00 -> 32.4 mm
- net CAN_RX: track 0.00 -> 29.8 mm
- net +5V: track 0.00 -> 28.1 mm
- net CAN_TX: track 0.00 -> 24.2 mm
- net CAN_EN: track 0.00 -> 22.4 mm, vias 0 -> 2
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
Commit message: Update PCB
Parts:
- removed J21: Conn_01x04, Connector_PinHeader_2.54mm:PinHeader_1x04_P2.54mm_Vertical
- C3, C4, C7: footprint Capacitor_THT:CP_Radial_D5.0mm_P2.50mm -> Capacitor_THT:C_Disc_D4.3mm_W1.9mm_P5.00mm
- J1, J14, J7: value Conn_01x02 -> Screw_Terminal_01x02; footprint Connector_PinHeader_2.54mm:PinHeader_1x02_P2.54mm_Vertical -> TerminalBlock_TE-Connectivity:TerminalBlock_TE_282834-2_1x02_P2.54mm_Horizontal
- J17, J18: value Conn_01x03 -> Screw_Terminal_01x03; footprint Connector_PinHeader_2.54mm:PinHeader_1x03_P2.54mm_Vertical -> TerminalBlock_TE-Connectivity:TerminalBlock_TE_282834-3_1x03_P2.54mm_Horizontal
- R10: footprint Resistor_THT:R_Axial_DIN0204_L3.6mm_D1.6mm_P7.62mm_Horizontal -> Resistor_THT:R_Axial_DIN0204_L3.6mm_D1.6mm_P2.54mm_Vertical
- moved J3 86.4 mm to (161.8, 88.5), turned to 90 degrees
- moved J19 73.2 mm to (161.5, 82.8), turned to 90 degrees
- moved J12 63.0 mm to (166.9, 112.0), turned to 270 degrees
- moved J13 61.1 mm to (159.2, 94.2), turned to 90 degrees
- moved J8 24.5 mm to (61.0, 95.0)
- moved BZ1 15.3 mm to (175.5, 103.8)
- moved J16 12.1 mm to (119.8, 145.5)
- moved J11 12.0 mm to (101.2, 145.5)
- moved J5 12.0 mm to (114.8, 145.5)
- moved J9 10.8 mm to (76.5, 111.8)
- moved C6 10.2 mm to (107.5, 138.2)
- moved J7 9.23 mm to (202.2, 95.7), turned to 270 degrees
- moved J1 9.20 mm to (202.2, 87.8), turned to 270 degrees
- moved J14 9.20 mm to (202.2, 103.2), turned to 270 degrees
- moved R1 9.20 mm to (195.2, 90.2)
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Connections:
- C2 pad 1: +5V -> Net-(C2-Pad1)
- J10 pad 1: Net-(J10-Pad1) -> Net-(C2-Pad1)
- J11 pad 2: GND -> GND_SCL
- J13 pad 1: GND -> /GND_232
- J19 pad 3: GND -> /GND_232
- J3 pad 4: GND -> /GND_232
- J5 pad 2: GND -> GND_SCL
- J8 pad 1: +5V -> Net-(C2-Pad1)
- J8 pad 2: +5V -> Net-(C2-Pad1)
- J8 pad 3: +5V -> Net-(C2-Pad1)
- J8 pad 4: +5V -> Net-(C2-Pad1)
- U1 pad 18: Net-(J10-Pad1) -> +5V
- U5 pad 3: +5V -> Net-(C2-Pad1)
Routing:
- net GND: track 56.9 -> 218.4 mm, vias 0 -> 4
- net door_sensor_1: track 7.02 -> 80.0 mm
- net door_sensor_3: track 7.02 -> 74.2 mm
- net door_sensor_2: track 7.02 -> 66.3 mm
- net buzz: track 0.00 -> 55.5 mm
- net Net-(J10-Pad1): track 34.9 -> 0.00 mm, vias 2 -> 0
- net /5V_micro: track 0.00 -> 33.0 mm, vias 0 -> 2
- net VCC: track 153.2 -> 124.6 mm, vias 0 -> 2
- net I2C_IRQ: track 0.00 -> 27.0 mm
- net /GND_232: track 0.00 -> 20.5 mm
- net +5V: track 28.1 -> 46.7 mm
- net GND_SCL: track 0.00 -> 16.7 mm
- net I2C_SCL: track 44.3 -> 29.4 mm
- net I2C_SDA: track 39.9 -> 25.3 mm
- net Net-(Q1-Pad2): track 6.68 -> 18.9 mm
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
Commit message: update PCB
Parts:
- removed J19: Conn_01x03, Connector_PinHeader_2.54mm:PinHeader_1x03_P2.54mm_Vertical
- removed J8, J9: Conn_01x04, Connector_PinHeader_2.54mm:PinHeader_1x04_P2.54mm_Vertical
- R10: footprint Resistor_THT:R_Axial_DIN0204_L3.6mm_D1.6mm_P2.54mm_Vertical -> Resistor_THT:R_Axial_DIN0207_L6.3mm_D2.5mm_P10.16mm_Horizontal
- moved R5 41.3 mm to (193.5, 64.5), turned to 270 degrees
- moved C4 38.4 mm to (189.0, 56.5), turned to 270 degrees
- moved C5 34.9 mm to (111.0, 94.5)
- moved R4 34.3 mm to (189.0, 64.5), turned to 270 degrees
- moved J5 33.7 mm to (119.0, 112.0)
- moved J11 33.6 mm to (119.0, 117.0)
- moved C6 33.5 mm to (112.0, 105.0)
- moved J10 33.0 mm to (114.0, 83.5), turned to 0 degrees
- moved D1 31.6 mm to (106.0, 76.1)
- moved BZ1 31.5 mm to (175.5, 72.3)
- moved J15 31.2 mm to (94.5, 72.5)
- moved J3 31.0 mm to (163.2, 57.5)
- moved J4 30.8 mm to (90.0, 95.8)
- moved J6 30.8 mm to (90.0, 107.2)
- moved R2 30.8 mm to (94.0, 91.8)
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Connections:
- J11 pad 1: VCC -> 3v3_I2C
- J5 pad 1: VCC -> 3v3_I2C
- U1 pad 20: VCC -> 3v3_I2C
Routing:
- net +5V: track 46.7 -> 182.5 mm, vias 0 -> 6
- net GND: track 218.4 -> 263.2 mm
- net door_sensor_3: track 74.2 -> 113.5 mm
- net door_sensor_2: track 66.3 -> 103.1 mm
- net /5V_micro: track 33.0 -> 0.00 mm, vias 2 -> 0
- net VCC: track 124.6 -> 156.3 mm
- net PN_RSTO: track 32.4 -> 57.2 mm
- net Net-(C2-Pad1): track 0.00 -> 21.9 mm
- net I2C_IRQ: track 27.0 -> 10.6 mm
- net door_sensor_1: track 80.0 -> 96.1 mm
- net 3v3_I2C: track 0.00 -> 12.5 mm
- net buzz: track 55.5 -> 47.3 mm
- net door_bell_1: track 38.1 -> 30.5 mm
- net door_bell_2: track 42.6 -> 35.7 mm
- net /Valt2: track 33.6 -> 29.2 mm
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Other:
- board outline added: 119 x 67 mm

Commit message: update PCB
Parts:
- added J8: Conn_01x04, Connector_PinHeader_2.54mm:PinHeader_1x04_P2.54mm_Vertical, F.Cu at (93.5, 117.3)
- added R14: 10k, Resistor_THT:R_Axial_DIN0207_L6.3mm_D2.5mm_P5.08mm_Vertical, F.Cu at (100.1, 110.5)
- added R15: 10k, Resistor_THT:R_Axial_DIN0207_L6.3mm_D2.5mm_P5.08mm_Vertical, F.Cu at (95.5, 113.8)
- moved C1 4.03 mm to (99.5, 80.8)
- moved C2 4.03 mm to (108.8, 81.0)
- moved J4 3.25 mm to (90.0, 92.5)
- moved J6 3.25 mm to (90.0, 104.0)
- moved R2 3.25 mm to (94.0, 88.5)
- moved R3 3.25 mm to (94.0, 100.0)
- moved R6 3.25 mm to (98.0, 87.5)
- moved R7 3.25 mm to (98.0, 99.0)
- moved U4 3.25 mm to (98.0, 90.5)
- moved U6 3.25 mm to (98.0, 102.0)
- moved U2 2.50 mm to (115.2, 64.5)
- moved C6 1.77 mm to (111.8, 103.3), turned to 180 degrees
- moved C5 1.50 mm to (111.0, 93.0)
- moved D2 1.50 mm to (175.0, 86.0)
- moved D1 1.25 mm to (106.0, 74.8)
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Connections:
- U1 pad 6: USART1_TX -> iButton_Data
- U1 pad 7: USART1_RX -> LED_iButton
Routing:
- net iButton_Data: track 0.00 -> 16.2 mm, vias 0 -> 1
- net VCC: track 156.3 -> 167.8 mm
- net I2C_IRQ: track 10.6 -> 21.1 mm, vias 0 -> 2
- net LED_iButton: track 0.00 -> 6.13 mm, vias 0 -> 1
- net /Valt1: track 16.5 -> 10.9 mm
- net GND: track 263.2 -> 267.2 mm
- net Net-(J8-Pad2): track 0.00 -> 3.72 mm
- net Net-(C1-Pad1): track 17.5 -> 14.9 mm
- net /CANL: track 5.88 -> 8.38 mm
- net /CANH: track 5.88 -> 8.38 mm
- net door_bell_2: track 35.7 -> 33.4 mm
- net CAN_TX: track 30.7 -> 28.8 mm
- net door_bell_1: track 30.5 -> 28.7 mm
- net CAN_EN: track 31.3 -> 32.9 mm
- net /Valt2: track 29.2 -> 27.9 mm
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
Commit message: PCB update
Routing:
- net LED_iButton: track 6.13 -> 52.8 mm
- net GND: track 267.2 -> 296.2 mm, vias 4 -> 6
- net door_sensor_1: track 96.1 -> 97.1 mm
- net buzz: track 46.4 -> 47.3 mm
Changed lines of the file:
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@@
     (thickness 1.6)
     (drawings 6)
-    (tracks 439)
+    (tracks 455)
     (zones 0)
     (modules 55)
@@
       (viasonmask false)
       (mode 1)
-      (useauxorigin false)
+      (useauxorigin true)
       (hpglpennumber 1)
       (hpglpenspeed 20)
@@
       (psnegative false)
       (psa4output false)
-      (plotreference true)
-      (plotvalue true)
+      (plotreference false)
+      (plotvalue false)
       (plotinvisibletext false)
       (padsonsilk false)
@@
   (segment (start 109.92 107.1) (end 111.75 105.27) (width 0.8) (layer B.Cu) (net 1))
   (segment (start 105.62 107.1) (end 109.92 107.1) (width 0.8) (layer B.Cu) (net 1))
+  (segment (start 184.5 56.52) (end 182.75 56.52) (width 0.8) (layer B.Cu) (net 1))
+  (via (at 180.71 62.37) (size 1.8) (drill 0.8) (layers F.Cu B.Cu) (net 1))
+  (segment (start 180.71 58.56) (end 180.71 62.37) (width 0.8) (layer B.Cu) (net 1))
+  (segment (start 182.75 56.52) (end 180.71 58.56) (width 0.8) (layer B.Cu) (net 1))
+  (via (at 184.52 77.61) (size 1.8) (drill 0.8) (layers F.Cu B.Cu) (net 1))
+  (segment (start 184.5 77.59) (end 184.52 77.61) (width 0.8) (layer B.Cu) (net 1))
+  (segment (start 184.5 74.68) (end 184.5 77.59) (width 0.8) (layer B.Cu) (net 1))
+  (segment (start 183.25 77.61) (end 184.52 77.61) (width 0.8) (layer F.Cu) (net 1))
+  (segment (start 180.71 75.07) (end 183.25 77.61) (width 0.8) (layer F.Cu) (net 1))
+  (segment (start 180.71 62.37) (end 180.71 75.07) (width 0.8) (layer F.Cu) (net 1))
   (segment (start 99.5 80.77) (end 99.83 80.77) (width 0.8) (layer B.Cu) (net 2))
   (segment (start 111.33 74.85) (end 111.5 75.02) (width 0.8) (layer B.Cu) (net 2))
@@
   (segment (start 126.61 64.41) (end 129 62.02) (width 0.8) (layer B.Cu) (net 4))
   (segment (start 126.27 64.41) (end 126.61 64.41) (width 0.8) (layer B.Cu) (net 4))
+  (segment (start 184.5 61.52) (end 184.5 62.52) (width 0.8) (layer B.Cu) (net 4))
   (segment (start 195.5 61.52) (end 196.5 62.52) (width 0.8) (layer B.Cu) (net 5))
   (segment (start 196.5 62.52) (end 196.5 65.52) (width 0.8) (layer B.Cu) (net 5))
@@
   (segment (start 127.49 72.03) (end 133.5 66.02) (width 0.8) (layer B.Cu) (net 66))
   (segment (start 126.27 72.03) (end 127.49 72.03) (width 0.8) (layer B.Cu) (net 66))
+  (segment (start 157.469 75.07) (end 156.58 75.07) (width 0.8) (layer B.Cu) (net 66))
   (segment (start 152 100.02) (end 152.5 99.52) (width 0.8) (layer B.Cu) (net 68))
   (segment (start 152.5 99.52) (end 155.5 99.52) (width 0.8) (layer B.Cu) (net 68))
@@
   (segment (start 121.38 79.65) (end 120.5 78.77) (width 0.8) (layer B.Cu) (net 79))
   (segment (start 126.27 79.65) (end 121.38 79.65) (width 0.8) (layer B.Cu) (net 79))
+  (segment (start 100.58 113.77) (end 106.45 113.77) (width 0.8) (layer F.Cu) (net 79))
+  (segment (start 106.45 113.77) (end 118.48 101.74) (width 0.8) (layer F.Cu) (net 79))
+  (segment (start 118.48 80.79) (end 120.5 78.77) (width 0.8) (layer F.Cu) (net 79))
+  (segment (start 118.48 101.74) (end 118.48 80.79) (width 0.8) (layer F.Cu) (net 79))
 )
