File: PCB/stm_proto_board_V2/stm_intercom_door_entrance.sch (KiCad schematic (older format))
At the start: 59 parts, among them J1 Screw_Terminal_01x02, J10 Conn_01x02, J11 Conn_01x04, J12 Conn_01x04, J13 Conn_01x04, J14 Screw_Terminal_01x02, J15 Conn_01x02, J16 Conn_01x01, J17 Screw_Terminal_01x03, J18 Screw_Terminal_01x03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

Commit message: update PCB
Connections:
- wire segments 203 -> 201
Other:
- moved on the sheet: J8, R14, R15
Changed lines of the file:
@@
 Wire Wire Line
 	4900 4800 4800 4800
+$Comp
+L power:+5V #PWR0119
+U 1 1 5B8AAD24
+P 4350 5200
+F 0 "#PWR0119" H 4350 5050 50  0001 C CNN
+F 1 "+5V" H 4365 5373 50  0000 C CNN
+F 2 "" H 4350 5200 50  0001 C CNN
+F 3 "" H 4350 5200 50  0001 C CNN
+	1    4350 5200
+	1    0    0    -1
+$EndComp
 Text Notes 6650 1450 0    50   ~ 0
 PN532 - I2C
@@
 Connection ~ 800  3100
 Connection ~ 1750 3100
+Wire Wire Line
+	4350 5200 4900 5200
 Wire Wire Line
 	4800 5300 4900 5300
@@
 L Connector_Generic:Conn_01x04 J8
 U 1 1 5FD87386
-P 3100 4450
-F 0 "J8" H 3180 4442 50  0000 L CNN
-F 1 "Conn_01x04" H 3180 4351 50  0000 L CNN
-F 2 "Connector_PinHeader_2.54mm:PinHeader_1x04_P2.54mm_Vertical" H 3100 4450 50  0001 C CNN
-F 3 "~" H 3100 4450 50  0001 C CNN
-	1    3100 4450
-	1    0    0    -1
-$EndComp
-Wire Wire Line
-	2900 4550 2800 4550
-Wire Wire Line
-	2800 4650 2900 4650
-Text Notes 2900 4900 0    50   ~ 0
+P 3100 4200
+F 0 "J8" H 3180 4192 50  0000 L CNN
+F 1 "Conn_01x04" H 3180 4101 50  0000 L CNN
+F 2 "Connector_PinHeader_2.54mm:PinHeader_1x04_P2.54mm_Vertical" H 3100 4200 50  0001 C CNN
+F 3 "~" H 3100 4200 50  0001 C CNN
+	1    3100 4200
+	1    0    0    -1
+$EndComp
+Wire Wire Line
+	2900 4100 2750 4100
+Wire Wire Line
+	2900 4300 2800 4300
+Wire Wire Line
+	2800 4400 2900 4400
+Text Notes 2900 4650 0    50   ~ 0
 iButton reader
-Text GLabel 2350 4450 0    50   Input ~ 0
+Wire Notes Line
+	3650 3800 3650 4700
+Text GLabel 2350 4200 0    50   Input ~ 0
 LED_iButton
-Text GLabel 2350 4350 0    50   Input ~ 0
+Text GLabel 2350 4100 0    50   Input ~ 0
 iButton_Data
 $Comp
 L power:GND #PWR0115
 U 1 1 5FDB1E01
-P 2800 4650
-F 0 "#PWR0115" H 2800 4400 50  0001 C CNN
-F 1 "GND" H 2805 4477 50  0000 C CNN
-F 2 "" H 2800 4650 50  0001 C CNN
-F 3 "" H 2800 4650 50  0001 C CNN
-	1    2800 4650
-	1    0    0    -1
-$EndComp
-Wire Wire Line
-	2800 4550 2800 4650
-Connection ~ 2800 4650
+P 2800 4400
+F 0 "#PWR0115" H 2800 4150 50  0001 C CNN
+F 1 "GND" H 2805 4227 50  0000 C CNN
+F 2 "" H 2800 4400 50  0001 C CNN
+F 3 "" H 2800 4400 50  0001 C CNN
+	1    2800 4400
+	1    0    0    -1
+$EndComp
+Wire Wire Line
+	2800 4300 2800 4400
+Connection ~ 2800 4400
 $Comp
 L Device:R R14
 U 1 1 5FE203BD
+P 2600 4100
+F 0 "R14" H 2670 4146 50  0000 L CNN
+F 1 "10k" H 2670 4055 50  0000 L CNN
+F 2 "Resistor_THT:R_Axial_DIN0207_L6.3mm_D2.5mm_P5.08mm_Vertical" V 2530 4100 50  0001 C CNN
+F 3 "~" H 2600 4100 50  0001 C CNN
+	1    2600 4100
+	0    -1   -1   0
+$EndComp
+$Comp
+L Device:R R15
+U 1 1 5FE2E898
 P 2600 4200
-F 0 "R14" H 2670 4246 50  0000 L CNN
+F 0 "R15" H 2670 4246 50  0000 L CNN
 F 1 "10k" H 2670 4155 50  0000 L CNN
 F 2 "Resistor_THT:R_Axial_DIN0207_L6.3mm_D2.5mm_P5.08mm_Vertical" V 2530 4200 50  0001 C CNN
 F 3 "~" H 2600 4200 50  0001 C CNN
 	1    2600 4200
-	0    -1   -1   0
-$EndComp
-$Comp
-L Device:R R15
-U 1 1 5FE2E898
-P 2600 4450
-F 0 "R15" H 2670 4496 50  0000 L CNN
-F 1 "10k" H 2670 4405 50  0000 L CNN
-F 2 "Resistor_THT:R_Axial_DIN0207_L6.3mm_D2.5mm_P5.08mm_Vertical" V 2530 4450 50  0001 C CNN
-F 3 "~" H 2600 4450 50  0001 C CNN
-	1    2600 4450
 	0    1    1    0
 $EndComp
 Wire Wire Line
-	2750 4450 2900 4450
-Wire Wire Line
-	2350 4450 2450 4450
-Wire Notes Line
-	1800 3950 3650 3950
-Wire Notes Line
-	1800 4950 3650 4950
+	2750 4200 2900 4200
+Wire Wire Line
+	2450 4100 2350 4100
+Wire Wire Line
+	2350 4200 2450 4200
+Wire Notes Line
+	1800 4700 1800 3800
+Wire Notes Line
+	1800 3800 3650 3800
+Wire Notes Line
+	1800 4700 3650 4700
 Wire Wire Line
 	800  2750 800  3000
@@
 Text GLabel 4750 4000 0    50   Input ~ 0
 iButton_Data
-Wire Wire Line
-	2350 4350 2750 4350
-Wire Wire Line
-	2750 4200 2750 4350
-Connection ~ 2750 4350
-Wire Wire Line
-	2750 4350 2900 4350
-Wire Wire Line
-	4350 5200 4900 5200
-$Comp
-L power:+5V #PWR0119
-U 1 1 5B8AAD24
-P 4350 5200
-F 0 "#PWR0119" H 4350 5050 50  0001 C CNN
-F 1 "+5V" H 4365 5373 50  0000 C CNN
-F 2 "" H 4350 5200 50  0001 C CNN
-F 3 "" H 4350 5200 50  0001 C CNN
-	1    4350 5200
-	1    0    0    -1
-$EndComp
-$Comp
-L power:+3V3 #PWR?
-U 1 1 5FDC5813
-P 2300 4200
-F 0 "#PWR?" H 2300 4050 50  0001 C CNN
-F 1 "+3V3" H 2315 4373 50  0000 C CNN
-F 2 "" H 2300 4200 50  0001 C CNN
-F 3 "" H 2300 4200 50  0001 C CNN
-	1    2300 4200
-	1    0    0    -1
-$EndComp
-Wire Wire Line
-	2450 4200 2300 4200
-Wire Notes Line
-	1800 3950 1800 4950
-Wire Notes Line
-	3650 3950 3650 4950
 $EndSCHEMATC
