File: PCB/stm_proto_board_V2/stm_proto_board.sch (KiCad schematic (older format))
At the start: 45 parts, among them J1 Conn_01x08, J10 Conn_01x02, J11 Conn_01x04, J12 Conn_01x04, J13 Conn_01x04, J14 Conn_01x08, J15 Conn_01x02, J16 Conn_01x03, J19 Conn_01x04, J2 Conn_01x04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

Commit message: Update schematic SDA/SDL pins
Parts:
- removed J5: Conn_01x04, Connector_PinHeader_2.54mm:PinHeader_1x04_P2.54mm_Vertical, symbol Connector_Generic:Conn_01x04
- added J17, J5: Conn_01x02, Connector_PinHeader_2.54mm:PinHeader_1x02_P2.54mm_Vertical, symbol Connector_Generic:Conn_01x02
- U3: symbol perso:MAX3232_convertor -> stm_proto_board-rescue:MAX3232_convertor-perso
Connections:
- wire segments 202 -> 201
Changed lines of the file:
@@
 Wire Wire Line
 	4950 4000 4800 4000
-Wire Wire Line
-	6550 3400 6750 3400
 Text GLabel 6650 3600 2    50   Input ~ 0
 USART3_RX
@@
 Wire Wire Line
 	10150 3450 9950 3450
-$Comp
-L Connector_Generic:Conn_01x04 J5
-U 1 1 5B81A704
-P 6700 1000
-F 0 "J5" H 6780 992 50  0000 L CNN
-F 1 "Conn_01x04" H 6780 901 50  0000 L CNN
-F 2 "Connector_PinHeader_2.54mm:PinHeader_1x04_P2.54mm_Vertical" H 6700 1000 50  0001 C CNN
-F 3 "~" H 6700 1000 50  0001 C CNN
-	1    6700 1000
-	1    0    0    -1
-$EndComp
-$Comp
-L power:+3V3 #PWR0115
-U 1 1 5B81E324
-P 6350 900
-F 0 "#PWR0115" H 6350 750 50  0001 C CNN
-F 1 "+3V3" H 6365 1073 50  0000 C CNN
-F 2 "" H 6350 900 50  0001 C CNN
-F 3 "" H 6350 900 50  0001 C CNN
-	1    6350 900
-	1    0    0    -1
-$EndComp
-$Comp
-L power:GND #PWR0117
-U 1 1 5B81E3CD
-P 6000 1200
-F 0 "#PWR0117" H 6000 950 50  0001 C CNN
-F 1 "GND" H 6005 1027 50  0000 C CNN
-F 2 "" H 6000 1200 50  0001 C CNN
-F 3 "" H 6000 1200 50  0001 C CNN
-	1    6000 1200
-	1    0    0    -1
-$EndComp
-Text GLabel 6400 1100 0    50   BiDi ~ 0
+Text GLabel 6400 1150 0    50   BiDi ~ 0
 SDA
-Text GLabel 6400 1200 0    50   Input ~ 0
+Text GLabel 6400 1250 0    50   Input ~ 0
 SCL
 Wire Wire Line
-	6500 900  6350 900
-Wire Wire Line
-	6000 1000 6000 1200
-Wire Wire Line
-	6000 1000 6500 1000
-Wire Wire Line
-	6500 1100 6400 1100
-Wire Wire Line
-	6400 1200 6500 1200
-Text GLabel 4850 4800 0    50   BiDi ~ 0
+	6500 1150 6400 1150
+Wire Wire Line
+	6400 1250 6500 1250
+Text GLabel 4800 4600 0    50   BiDi ~ 0
 SDA
 Wire Wire Line
 	4950 4800 4850 4800
-Text GLabel 4850 4700 0    50   Output ~ 0
+Text GLabel 4800 4500 0    50   Output ~ 0
 SCL
 Wire Wire Line
 	4950 4700 4850 4700
-Text GLabel 4800 4600 0    50   Input ~ 0
+Text GLabel 4850 4800 0    50   Input ~ 0
 SW_DOWN
-Text GLabel 4800 4500 0    50   Input ~ 0
+Text GLabel 4850 4700 0    50   Input ~ 0
 SW_RIGHT
 Text GLabel 4800 4300 0    50   Input ~ 0
@@
 $EndComp
 $Comp
-L perso:MAX3232_convertor U3
+L stm_proto_board-rescue:MAX3232_convertor-perso U3
 U 1 1 5B6FB7F9
 P 8800 3200
@@
 $EndComp
 Wire Wire Line
-	6750 3400 6750 3250
-$Comp
-L power:+3V3 #PWR0118
-U 1 1 5B89DD8A
-P 6750 3250
-F 0 "#PWR0118" H 6750 3100 50  0001 C CNN
-F 1 "+3V3" H 6765 3423 50  0000 C CNN
-F 2 "" H 6750 3250 50  0001 C CNN
-F 3 "" H 6750 3250 50  0001 C CNN
-	1    6750 3250
-	1    0    0    -1
-$EndComp
-Wire Wire Line
 	1850 4550 2350 4550
 $Comp
@@
 	1    0    0    -1
 $EndComp
+$Comp
+L Connector_Generic:Conn_01x02 J5
+U 1 1 5FABC2C9
+P 6700 900
+F 0 "J5" H 6780 892 50  0000 L CNN
+F 1 "Conn_01x02" H 6780 801 50  0000 L CNN
+F 2 "Connector_PinHeader_2.54mm:PinHeader_1x02_P2.54mm_Vertical" H 6700 900 50  0001 C CNN
+F 3 "~" H 6700 900 50  0001 C CNN
+	1    6700 900
+	1    0    0    -1
+$EndComp
+$Comp
+L Connector_Generic:Conn_01x02 J17
+U 1 1 5FAE99A1
+P 6700 1150
+F 0 "J17" H 6780 1142 50  0000 L CNN
+F 1 "Conn_01x02" H 6780 1051 50  0000 L CNN
+F 2 "Connector_PinHeader_2.54mm:PinHeader_1x02_P2.54mm_Vertical" H 6700 1150 50  0001 C CNN
+F 3 "~" H 6700 1150 50  0001 C CNN
+	1    6700 1150
+	1    0    0    -1
+$EndComp
+Wire Wire Line
+	6750 3400 6750 3250
+Wire Wire Line
+	6550 3400 6750 3400
+$Comp
+L power:+3V3 #PWR0118
+U 1 1 5B89DD8A
+P 6750 3250
+F 0 "#PWR0118" H 6750 3100 50  0001 C CNN
+F 1 "+3V3" H 6765 3423 50  0000 C CNN
+F 2 "" H 6750 3250 50  0001 C CNN
+F 3 "" H 6750 3250 50  0001 C CNN
+	1    6750 3250
+	1    0    0    -1
+$EndComp
+$Comp
+L power:+3V3 #PWR0115
+U 1 1 5B81E324
+P 6350 900
+F 0 "#PWR0115" H 6350 750 50  0001 C CNN
+F 1 "+3V3" H 6365 1073 50  0000 C CNN
+F 2 "" H 6350 900 50  0001 C CNN
+F 3 "" H 6350 900 50  0001 C CNN
+	1    6350 900
+	1    0    0    -1
+$EndComp
+Wire Wire Line
+	6500 900  6350 900
+Text GLabel 6350 1000 0    50   Input ~ 0
+GND_SCL
+Wire Wire Line
+	6350 1000 6500 1000
 Wire Bus Line
 	4300 3300 4300 5250

Commit message: Update schematic
Connections:
- net labels added: 3.3v_teleinfo
- wire segments 201 -> 198
Other:
- note added: "Control switches"
- note added: "PN532 - I2C"
- note removed: "PN532"
- moved on the sheet: C1, C2, D1, J8, J9, R6, U5

Commit message: update schematics
Parts:
- added BZ1: Buzzer, Buzzer_Beeper:Buzzer_12x9.5RM7.6, symbol Device:Buzzer
- added J18: Conn_01x03, Connector_PinHeader_2.54mm:PinHeader_1x03_P2.54mm_Vertical, symbol Connector_Generic:Conn_01x03
- added R13: 330, Resistor_THT:R_Axial_DIN0204_L3.6mm_D1.6mm_P7.62mm_Horizontal, symbol Device:R
Connections:
- net labels added: CANH, CANL, TP10, TP8, TP9, buzz
- net labels removed: Ext11, Ext12, Ext8, Ext9
Other:
- note added: "Buzzer"

Commit message: update PCB
Parts:
- removed J3: DB9_Female, Connector_Dsub:DSUB-9_Female_Horizontal_P2.77x2.84mm_EdgePinOffset4.94mm_Housed_MountingHolesOffset7.48mm, symbol Connector:DB9_Female
- added J20, J3: Conn_01x04, Connector_PinHeader_2.54mm:PinHeader_1x04_P2.54mm_Vertical, symbol Connector_Generic:Conn_01x04
- added R14, R15: 330, Resistor_THT:R_Axial_DIN0204_L3.6mm_D1.6mm_P7.62mm_Horizontal, symbol Device:R
- added RV1: R_POT, Potentiometer_THT:Potentiometer_Bourns_3266Z_Horizontal, symbol Device:R_POT
- R5: footprint Resistor_THT:R_Axial_DIN0204_L3.6mm_D1.6mm_P7.62mm_Horizontal -> Resistor_THT:R_Axial_DIN0204_L3.6mm_D1.6mm_P5.08mm_Horizontal
- U5: footprint Package_TO_SOT_THT:TO-220-3_Vertical -> Package_TO_SOT_THT:TO-220-3_Horizontal_TabUp
Connections:
- net labels added: GND_232, RS232_GND, RS232_RX, RS232_TX, ibutton_data, ibutton_led+
- wire segments 198 -> 201
Other:
- note added: "Wires color:\n1. red\n2. white\n3. black\n4. green"
- note added: "ibutton reader"
- moved on the sheet: J12, J13, J16, J18, J19, J4, R10, R11, R12, R5, R6, R7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

Commit message: update PCB
Connections:
- net TP1: no longer U1.6 (PA9)
- net TP2: no longer U1.7 (PA10)
- net ibutton_data: now also U1.6 (PA9)
- net ibutton_led+: now also U1.7 (PA10)
Changed lines of the file:
@@
 Text GLabel 4750 4100 0    50   Output ~ 0
 TP3
-Text GLabel 4750 3800 0    50   Output ~ 0
+Text GLabel 4100 3500 0    50   Output ~ 0
 TP2
-Text GLabel 4750 3700 0    50   Output ~ 0
+Text GLabel 4100 3400 0    50   Output ~ 0
 TP1
 Wire Wire Line
@@
 Wire Wire Line
 	4750 4100 4950 4100
-Wire Wire Line
-	4750 3800 4950 3800
-Wire Wire Line
-	4950 3700 4750 3700
 Wire Wire Line
 	4750 3600 4950 3600
@@
 Wire Wire Line
 	1050 4850 1150 4850
-$Comp
-L Connector_Generic:Conn_01x04 J20
-U 1 1 5FB0F0D0
-P 9850 6000
-F 0 "J20" H 9930 5992 50  0000 L CNN
-F 1 "Conn_01x04" H 9930 5901 50  0000 L CNN
-F 2 "Connector_PinHeader_2.54mm:PinHeader_1x04_P2.54mm_Vertical" H 9850 6000 50  0001 C CNN
-F 3 "~" H 9850 6000 50  0001 C CNN
-	1    9850 6000
-	1    0    0    -1
-$EndComp
-Text GLabel 9250 6200 0    50   Input ~ 0
+Text GLabel 4850 3700 0    50   Input ~ 0
+ibutton_data
+Text GLabel 4850 3800 0    50   Input ~ 0
 ibutton_led+
-Text GLabel 9500 5900 0    50   Input ~ 0
-ibutton_data
-Wire Wire Line
-	9650 5900 9550 5900
-Text Notes 10500 6200 0    50   ~ 0
-Wires color:\n1. red\n2. white\n3. black\n4. green
-$Comp
-L power:GND #PWR0117
-U 1 1 5FBB0AC2
-P 9650 6200
-F 0 "#PWR0117" H 9650 5950 50  0001 C CNN
-F 1 "GND" H 9655 6027 50  0000 C CNN
-F 2 "" H 9650 6200 50  0001 C CNN
-F 3 "" H 9650 6200 50  0001 C CNN
-	1    9650 6200
-	1    0    0    -1
-$EndComp
-Text Notes 10400 6400 0    50   ~ 0
-ibutton reader
-$Comp
-L Device:R R14
-U 1 1 5FB24111
-P 9250 5800
-F 0 "R14" V 9043 5800 50  0000 C CNN
-F 1 "330" V 9134 5800 50  0000 C CNN
-F 2 "Resistor_THT:R_Axial_DIN0204_L3.6mm_D1.6mm_P7.62mm_Horizontal" V 9180 5800 50  0001 C CNN
-F 3 "~" H 9250 5800 50  0001 C CNN
-	1    9250 5800
-	0    1    1    0
-$EndComp
-Wire Wire Line
-	9550 5800 9550 5900
-Connection ~ 9550 5900
-Wire Wire Line
-	9550 5900 9500 5900
-Wire Wire Line
-	9400 5800 9550 5800
-Wire Notes Line
-	11000 5550 11000 6450
-Wire Notes Line
-	8650 5550 8650 6450
-Wire Notes Line
-	8650 5550 11000 5550
-Wire Notes Line
-	8650 6450 11000 6450
-Text GLabel 7100 5150 2    50   Input ~ 0
-ibutton_data
-Text GLabel 7100 5300 2    50   Input ~ 0
-ibutton_led+
-Wire Wire Line
-	9650 6100 9650 6200
-Connection ~ 9650 6200
-$Comp
-L Device:R R15
-U 1 1 5FD3DA1B
-P 9400 6200
-F 0 "R15" V 9193 6200 50  0000 C CNN
-F 1 "330" V 9284 6200 50  0000 C CNN
-F 2 "Resistor_THT:R_Axial_DIN0204_L3.6mm_D1.6mm_P7.62mm_Horizontal" V 9330 6200 50  0001 C CNN
-F 3 "~" H 9400 6200 50  0001 C CNN
-	1    9400 6200
-	0    1    1    0
-$EndComp
-Wire Wire Line
-	9550 6200 9550 6000
-Wire Wire Line
-	9550 6000 9650 6000
-$Comp
-L power:+3.3V #PWR0118
-U 1 1 5FDDA0F7
-P 8900 5800
-F 0 "#PWR0118" H 8900 5650 50  0001 C CNN
-F 1 "+3.3V" H 8915 5973 50  0000 C CNN
-F 2 "" H 8900 5800 50  0001 C CNN
-F 3 "" H 8900 5800 50  0001 C CNN
-	1    8900 5800
-	1    0    0    -1
-$EndComp
-Wire Wire Line
-	8900 5800 9100 5800
 Wire Wire Line
 	9600 3750 9950 3750
@@
 Text Label 9400 3000 0    50   ~ 0
 RS232_TX
+Wire Wire Line
+	8900 5800 9100 5800
+$Comp
+L power:+3.3V #PWR0118
+U 1 1 5FDDA0F7
+P 8900 5800
+F 0 "#PWR0118" H 8900 5650 50  0001 C CNN
+F 1 "+3.3V" H 8915 5973 50  0000 C CNN
+F 2 "" H 8900 5800 50  0001 C CNN
+F 3 "" H 8900 5800 50  0001 C CNN
+	1    8900 5800
+	1    0    0    -1
+$EndComp
+Wire Wire Line
+	9550 6000 9650 6000
+Wire Wire Line
+	9550 6200 9550 6000
+$Comp
+L Device:R R15
+U 1 1 5FD3DA1B
+P 9400 6200
+F 0 "R15" V 9193 6200 50  0000 C CNN
+F 1 "330" V 9284 6200 50  0000 C CNN
+F 2 "Resistor_THT:R_Axial_DIN0204_L3.6mm_D1.6mm_P7.62mm_Horizontal" V 9330 6200 50  0001 C CNN
+F 3 "~" H 9400 6200 50  0001 C CNN
+	1    9400 6200
+	0    1    1    0
+$EndComp
+Connection ~ 9650 6200
+Wire Wire Line
+	9650 6100 9650 6200
+Wire Notes Line
+	8650 6450 11000 6450
+Wire Notes Line
+	8650 5550 11000 5550
+Wire Notes Line
+	8650 5550 8650 6450
+Wire Notes Line
+	11000 5550 11000 6450
+Wire Wire Line
+	9400 5800 9550 5800
+Wire Wire Line
+	9550 5900 9500 5900
+Connection ~ 9550 5900
+Wire Wire Line
+	9550 5800 9550 5900
+$Comp
+L Device:R R14
+U 1 1 5FB24111
+P 9250 5800
+F 0 "R14" V 9043 5800 50  0000 C CNN
+F 1 "330" V 9134 5800 50  0000 C CNN
+F 2 "Resistor_THT:R_Axial_DIN0204_L3.6mm_D1.6mm_P7.62mm_Horizontal" V 9180 5800 50  0001 C CNN
+F 3 "~" H 9250 5800 50  0001 C CNN
+	1    9250 5800
+	0    1    1    0
+$EndComp
+Text Notes 10400 6400 0    50   ~ 0
+ibutton reader
+$Comp
+L power:GND #PWR0117
+U 1 1 5FBB0AC2
+P 9650 6200
+F 0 "#PWR0117" H 9650 5950 50  0001 C CNN
+F 1 "GND" H 9655 6027 50  0000 C CNN
+F 2 "" H 9650 6200 50  0001 C CNN
+F 3 "" H 9650 6200 50  0001 C CNN
+	1    9650 6200
+	1    0    0    -1
+$EndComp
+Text Notes 10500 6200 0    50   ~ 0
+Wires color:\n1. red\n2. white\n3. black\n4. green
+Wire Wire Line
+	9650 5900 9550 5900
+Text GLabel 9500 5900 0    50   Input ~ 0
+ibutton_data
+Text GLabel 9250 6200 0    50   Input ~ 0
+ibutton_led+
+$Comp
+L Connector_Generic:Conn_01x04 J20
+U 1 1 5FB0F0D0
+P 9850 6000
+F 0 "J20" H 9930 5992 50  0000 L CNN
+F 1 "Conn_01x04" H 9930 5901 50  0000 L CNN
+F 2 "Connector_PinHeader_2.54mm:PinHeader_1x04_P2.54mm_Vertical" H 9850 6000 50  0001 C CNN
+F 3 "~" H 9850 6000 50  0001 C CNN
+	1    9850 6000
+	1    0    0    -1
+$EndComp
+Wire Wire Line
+	4950 3800 4850 3800
+Wire Wire Line
+	4850 3700 4950 3700
 Wire Bus Line
 	4300 3300 4300 5250

Commit message: Update PCB proto board
Parts:
- BZ1: symbol Device:Buzzer -> stm_proto_board-rescue:Buzzer-Device
- C1, C2: symbol pspice:CAP -> stm_proto_board-rescue:CAP-pspice
- D1: symbol Device:D_Bridge_+-AA -> stm_proto_board-rescue:D_Bridge_+-AA-Device
- J1, J14: symbol Connector_Generic:Conn_01x08 -> stm_proto_board-rescue:Conn_01x08-Connector_Generic
- J10, J15, J17, J4, J5, J6: symbol Connector_Generic:Conn_01x02 -> stm_proto_board-rescue:Conn_01x02-Connector_Generic
- J11, J12, J13, J19, J2, J20, J3, J7, J8, J9: symbol Connector_Generic:Conn_01x04 -> stm_proto_board-rescue:Conn_01x04-Connector_Generic
- J16, J18: symbol Connector_Generic:Conn_01x03 -> stm_proto_board-rescue:Conn_01x03-Connector_Generic
- R1, R10, R11, R12, R13, R14, R15, R2, R3, R4, R5, R6, R7, R8, R9: symbol Device:R -> stm_proto_board-rescue:R-Device
- RV1: symbol Device:R_POT -> stm_proto_board-rescue:R_POT-Device
- SW1, SW2, SW3, SW4: symbol Switch:SW_Push -> stm_proto_board-rescue:SW_Push-Switch
- U2: symbol Interface_CAN_LIN:MCP2551-I-P -> stm_proto_board-rescue:MCP2551-I-P-Interface_CAN_LIN
- U4: symbol Isolator:LTV-814 -> stm_proto_board-rescue:LTV-814-Isolator
- U5: symbol Regulator_Linear:L7805 -> stm_proto_board-rescue:L7805-Regulator_Linear
- U6, U7, U8, U9: symbol Isolator:4N25 -> stm_proto_board-rescue:4N25-Isolator
Connections:
- net TP1 is gone; now on net ibutton_data: J16.1 (Pin_1)
- net TP2 is gone; now on net ibutton_led+: J16.2 (Pin_2)
- no-connect marks 0 -> 18
Other:
- moved on the sheet: J16, J18, J19
