File: PCB/stm_proto_board_V2/stm_proto_board.kicad_pcb (KiCad board)
At the start: 2 copper layers, 137.2 x 81.3 mm, 43 parts, among them J1 Conn_01x08, J10 Conn_01x02, J11 Conn_01x04, J12 Conn_01x04, J13 Conn_01x04, J14 Conn_01x08, J15 Conn_01x02, J16 Conn_01x03, J19 Conn_01x04, J2 Conn_01x04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

Commit message: Update schematic SDA/SDL pins
Parts:
- removed J11: Conn_01x04, Connector_PinHeader_2.54mm:PinHeader_1x04_P2.54mm_Vertical
- added J17: Conn_01x02, Connector_PinHeader_2.54mm:PinHeader_1x02_P2.54mm_Vertical, F.Cu at (151.1, 96.5)
- added J5: Conn_01x02, Connector_PinHeader_2.54mm:PinHeader_1x02_P2.54mm_Vertical, F.Cu at (163.8, 97.8)
Connections:
- U1 pad 14: SW_RIGHT -> SCL
- U1 pad 15: SW_DOWN -> SDA
- U1 pad 16: SCL -> SW_RIGHT
- U1 pad 17: SDA -> SW_DOWN
Routing:
- net SW_RIGHT: track 28.5 -> 32.1 mm
- net SCL: track 8.67 -> 6.35 mm
- net SDA: track 8.67 -> 6.35 mm
- net SW_DOWN: track 45.7 -> 46.8 mm

Commit message: Update schematic
Parts:
- added J11: Conn_01x04, Connector_PinHeader_2.54mm:PinHeader_1x04_P2.54mm_Vertical, F.Cu at (203.0, 110.0)
- moved J12 21.0 mm to (191.2, 120.7), turned to 270 degrees
- moved C2 20.2 mm to (87.6, 104.1)
- moved C1 18.9 mm to (90.2, 115.6)
- moved U5 13.1 mm to (90.2, 124.5)
- moved J10 13.0 mm to (81.3, 100.3)
- moved J8 13.0 mm to (81.3, 118.1)
- moved J9 7.63 mm to (140.0, 138.0), turned to 180 degrees
- moved J13 6.93 mm to (183.6, 138.5), turned to 90 degrees
- moved J2 2.54 mm to (88.9, 81.3)
- moved U2 2.54 mm to (102.9, 81.3)
- moved J4 1.27 mm to (210.8, 73.7)
- moved R5 1.27 mm to (207.0, 73.7)
- moved R12 1.27 mm to (119.4, 111.8)
- moved U4 1.27 mm to (195.6, 73.7)
Connections:
- R6 pad 1: +3V3 -> 3.3v_teleinfo
- U1 pad 38: +3V3 -> 3.3v_teleinfo
Routing:
- net USART2_TX: track 112.2 -> 89.7 mm
- net +3V3: track 225.3 -> 242.3 mm
- net GND: track 421.6 -> 404.8 mm, vias 9 -> 7
- net USART2_RX: track 114.0 -> 98.2 mm
- net Net-(J13-Pad1): track 10.6 -> 25.1 mm
- net Net-(C1-Pad1): track 38.5 -> 27.0 mm
- net Net-(J13-Pad3): track 10.8 -> 22.0 mm
- net CAN_RX: track 40.7 -> 51.1 mm, vias 2 -> 0
- net Net-(J13-Pad4): track 10.9 -> 18.3 mm
- net 3.3v_teleinfo: track 0.00 -> 6.88 mm
- net +5V: track 34.9 -> 40.5 mm
- net Net-(J10-Pad1): track 130.9 -> 126.5 mm
- net /Valt2: track 30.8 -> 33.3 mm
- net /Valt1: track 18.1 -> 20.6 mm
- net CAN_EN: track 34.6 -> 37.1 mm
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
Commit message: update schematics
Parts:
- added BZ1: Buzzer, Buzzer_Beeper:Buzzer_12x9.5RM7.6, F.Cu at (172.4, 71.0)
- added J18: Conn_01x03, Connector_PinHeader_2.54mm:PinHeader_1x03_P2.54mm_Vertical, F.Cu at (134.0, 68.5)
- added R13: 330, Resistor_THT:R_Axial_DIN0204_L3.6mm_D1.6mm_P7.62mm_Horizontal, F.Cu at (168.5, 68.0)
- moved R12 5.32 mm to (123.3, 108.1), turned to 270 degrees
- moved R11 0.18 mm to (119.5, 108.1), turned to 270 degrees
Connections:
- net Net-(J2-Pad2) renamed /CANH
- net Net-(J2-Pad3) renamed /CANL
- U1 pad 26: Ext8 -> buzz
- U1 pad 29: Ext9 -> TP10
- U1 pad 34: Ext11 -> TP9
- U1 pad 35: Ext12 -> TP8
Routing:
- net buzz: track 0.00 -> 24.4 mm, vias 0 -> 1
- net TP9: track 0.00 -> 10.9 mm
- net TP8: track 0.00 -> 9.98 mm
- net TP10: track 0.00 -> 8.26 mm
- net Net-(BZ1-Pad1): track 0.00 -> 5.14 mm
- net USART2_RX: track 98.2 -> 103.2 mm
- net +3V3: track 242.3 -> 244.1 mm
- net GND: track 404.8 -> 403.3 mm
- net USART2_TX: track 89.7 -> 90.5 mm
- net USART3_RX: track 73.8 -> 74.6 mm

Commit message: update PCB
Parts:
- added J20: Conn_01x04, Connector_PinHeader_2.54mm:PinHeader_1x04_P2.54mm_Vertical, F.Cu at (167.4, 138.6)
- added R14: 330, Resistor_THT:R_Axial_DIN0204_L3.6mm_D1.6mm_P7.62mm_Horizontal, F.Cu at (167.5, 133.3)
- added R15: 330, Resistor_THT:R_Axial_DIN0204_L3.6mm_D1.6mm_P7.62mm_Horizontal, F.Cu at (171.4, 130.2)
- added RV1: R_POT, Potentiometer_THT:Potentiometer_Bourns_3266Z_Horizontal, F.Cu at (120.1, 126.0)
- J3: value DB9_Female -> Conn_01x04; footprint Connector_Dsub:DSUB-9_Female_Horizontal_P2.77x2.84mm_EdgePinOffset4.94mm_Housed_MountingHolesOffset7.48mm -> Connector_PinHeader_2.54mm:PinHeader_1x04_P2.54mm_Vertical
- R5: footprint Resistor_THT:R_Axial_DIN0204_L3.6mm_D1.6mm_P7.62mm_Horizontal -> Resistor_THT:R_Axial_DIN0204_L3.6mm_D1.6mm_P5.08mm_Horizontal
- U5: footprint Package_TO_SOT_THT:TO-220-3_Vertical -> Package_TO_SOT_THT:TO-220-3_Horizontal_TabUp
- moved J8 23.0 mm to (98.3, 133.6), turned to 270 degrees
- moved U5 17.3 mm to (107.4, 122.9), turned to 270 degrees
- moved C1 10.5 mm to (100.1, 112.1), turned to 270 degrees
- moved J7 10.3 mm to (204.0, 92.8), turned to 180 degrees
- moved R11 10.3 mm to (120.1, 118.4), turned to 90 degrees
- moved J10 9.73 mm to (88.6, 94.0)
- moved C2 8.70 mm to (88.6, 112.8)
- moved R5 7.33 mm to (200.9, 77.7)
- moved J6 7.08 mm to (204.0, 103.4), turned to 0 degrees
- moved J15 6.71 mm to (94.7, 86.9), turned to 270 degrees
- moved J4 6.35 mm to (204.5, 73.7)
- moved J11 5.16 mm to (198.0, 111.3), turned to 0 degrees
- moved J3 3.82 mm to (198.0, 126.7), turned to 0 degrees
- moved U8 3.05 mm to (192.5, 86.4)
- moved U9 3.05 mm to (192.5, 97.8)
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Connections:
- net Net-(J13-Pad4) renamed /RS232_TX
- J13 pad 1: Net-(J13-Pad1) -> /RS232_GND
- J13 pad 2: Net-(J13-Pad2) -> /GND_232
- J13 pad 3: Net-(J13-Pad3) -> /RS232_RX
- J3 pad 1: Net-(J3-Pad1) -> /RS232_RX
- J3 pad 3: Net-(J13-Pad3) -> Net-(J3-Pad3)
- J3 pad 4: Net-(J3-Pad4) -> /GND_232
- J6 pad 1: OUT_W -> GND
- J6 pad 2: GND -> OUT_W
- J7 pad 1: OUT_R -> GND
- J7 pad 2: OUT_G -> OUT_B
- J7 pad 3: OUT_B -> OUT_G
- J7 pad 4: GND -> OUT_R
- R11 pad 1: /LIGHT -> Net-(R11-Pad1)
- R12 pad 2: /LIGHT -> Net-(R12-Pad2)
Routing:
- net GND: track 403.3 -> 433.6 mm, vias 7 -> 8
- net Net-(J13-Pad1): track 25.1 -> 0.00 mm
- net +5V: track 40.5 -> 63.6 mm
- net Net-(J13-Pad3): track 22.0 -> 0.00 mm
- net /GND_232: track 0.00 -> 19.9 mm
- net Net-(J10-Pad1): track 126.5 -> 107.7 mm
- net /RS232_RX: track 0.00 -> 17.9 mm
- net /Valt2: track 33.3 -> 21.5 mm
- net Net-(J20-Pad2): track 0.00 -> 9.01 mm
- net OUT_W: track 32.4 -> 23.7 mm
- net /LIGHT: track 17.0 -> 25.1 mm
- net Net-(R12-Pad2): track 0.00 -> 7.62 mm
- net Net-(R11-Pad1): track 0.00 -> 7.62 mm
- net /Valt1: track 20.6 -> 13.3 mm
- net +3V3: track 244.1 -> 251.3 mm
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Other:
- board size 137.2 x 81.3 mm -> 120.9 x 78.2 mm
- board text added: "+5V"
- board text added: "GND"
- board text added: "I2C"
- board text added: "RS232"
- board text added: "ibutton"

Commit message: Update PCB proto board
Connections:
- J16 pad 1: TP1 -> ibutton_data
- J16 pad 2: TP2 -> ibutton_led+
- U1 pad 6: TP1 -> ibutton_data
- U1 pad 7: TP2 -> ibutton_led+
Routing:
- net ibutton_led+: track 0.00 -> 87.4 mm
- net ibutton_data: track 5.26 -> 81.8 mm
- net SCL: track 6.35 -> 79.5 mm
- net SDA: track 6.35 -> 79.4 mm
- net GND_SCL: track 7.62 -> 55.0 mm
- net +3V3: track 251.3 -> 271.0 mm
- net TP2: track 6.35 -> 0.00 mm
- net TP1: track 6.35 -> 0.00 mm
- net GND: track 433.6 -> 436.1 mm
- net USART2_TX: track 90.5 -> 88.4 mm
- net USART2_RX: track 103.2 -> 101.7 mm
Other:
- board text added: "STM Proto board v2"
- board text added: "iButton"
- board text removed: "ibutton"
